File: dap/adau1467.kicad_sch (KiCad schematic)
At the start: 2 parts, among them U1 SI53301-B-GM, U2 ADAU1467WBCPZ300

Commit message: general setup
Parts:
- added C? (x3): 10u, symbol Device:C_Small
- added C? (x3): 10u, symbol Device:C_Polarized_Small
- added C? (x2): .1u, symbol Device:C_Small
- added C?: 100u, symbol Device:C_Polarized_Small
- added C? (x2): 1u, symbol Device:C_Small
- added D?: Green LED, symbol Device:LED_Small_Filled
- added FB?: FerriteBead, symbol Device:FerriteBead
- added J?: Conn_02x05_Odd_Even, symbol Connector_Generic:Conn_02x05_Odd_Even
- added Q?: STD2805T4, hf-transceiver:DPAKTO-252_TYPEA_STM, symbol hf-transceiver:STD2805T4
- added R15, R?: 1k, symbol Device:R_Small_US
- added R?: 0.47, symbol Device:R_Small_US
- added R? (x3): 10k, symbol Device:R_Small_US
- added R?: ?, symbol Device:R_Small_US
- added R?: 0, symbol Device:R_Small_US
- added R?: 100k, symbol Device:R_Small_US
- added SW? (x2): SW_Push, symbol Switch:SW_Push
- added TP?: TestPoint, symbol Connector:TestPoint_Probe
- added U?: ADM811TARTZ-REEL7, hf-transceiver:RA_4_ADI, symbol hf-transceiver:ADM811TARTZ-REEL7
- added U?: ADP3338, Package_TO_SOT_SMD:SOT-223, symbol hf-transceiver:ADP3338
- added U?: 25AA1024-I/MF, DFN-S8_6x5MC_MCH, symbol hf-transceiver:25AA1024-I_MF
Connections:
- new net: C?.2, R?.1
- new net: R?.2, SW?.1, U?.3 (MR*)
- new net: R?.2, U?.3 (*WP)
- new net: Q?.3 (Emitter), R15.1
- new net: Q?.1 (Base), R15.2
- new net: D?.2 (A), R?.2
- new net +5V: C?.1, C?.2, J?.4 (Pin_4), R?.1, U?.3 (In)
- new net AVDD: C?.1, C?.2, C?.2, FB?.1, R?.2, TP?.1, U?.2 (Out), U?.4 (Out)
- new net DVDD: C?.1, Q?.2 (Collector)
- new net GND: C?.1, C?.1, C?.1, C?.1, C?.1, C?.1, C?.2, C?.2, C?.2, C?.2, D?.1 (K), J?.10 (Pin_10), R?.2, R?.2, SW?.2, U?.1 (GND), U?.1 (GND), U?.4 (VSS)
- new net IOVDD: C?.1, C?.1, C?.2, C?.2, FB?.2, R?.1, R?.1, R?.1, SW?.1, U?.4 (VCC), U?.7 (*HOLD), U?.8 (VCC)
- new net MISO: J?.5 (Pin_5)
- new net MOSI: J?.8 (Pin_8)
- new net MOSI_M/MP1: U?.5 (SI)
- new net MiSO_M: U?.2 (SO)
- new net PVDD: C?.2, R?.1
- new net SCL: J?.1 (Pin_1)
- new net SCLCK: J?.7 (Pin_7)
- new net SCLK_M: U?.6 (SCK)
- new net SDA: J?.3 (Pin_3)
- new net SELFBOOT: SW?.2
- new net SS: J?.9 (Pin_9), R?.2
- new net SS_M/MP0: R?.2, U?.1 (*CS)
- new net USB_~{RESET}: J?.6 (Pin_6), R?.1
- new net ~{RESET}: R?.1, U?.2 (RESET*)
- no-connect marks 0 -> 1
Other:
- note added: "600 ohms at 100MHz"
- note added: "DVDD Regulator Circuit"
- note added: "Eval Board Scheamtic Quick Access"
- note added: "Going to need to properly source this"
- note added: "Power Supply Bulk Decoupling"
- note added: "Reset Circuit"
- note added: "SPI 10 Pin Connector"
- note added: "Self Boot Circuit"
- moved on the sheet: U1, U2A, U2B
