File: dap/tx_mixers.kicad_sch (KiCad schematic)
At the start: 2 parts, among them U10 SN74CBT3253, U9 SN74CBT3253

Commit message: general setup
Parts:
- removed U10, U9: SN74CBT3253, symbol Analog_Switch:SN74CBT3253
- added C21, C22: 47u, Capacitor_SMD:C_0805_2012Metric_Pad1.18x1.45mm_HandSolder, symbol Device:C_Polarized_Small_US
- added C23, C24, C25, C26, C27, C28, C29, C30, C31, C32: 0.1u, Capacitor_SMD:C_0805_2012Metric_Pad1.18x1.45mm_HandSolder, symbol Device:C_Small
- added C33, C34, C35, C36, C37, C38, C39, C40: 0.068u, Capacitor_SMD:C_0805_2012Metric_Pad1.18x1.45mm_HandSolder, symbol Device:C_Small
- added H5, H6, H7, H8: MountingHole, MountingHole:MountingHole_3.2mm_M3, symbol Mechanical:MountingHole
- added J23: Conn_01x05_Pin, Connector_PinHeader_2.54mm:PinHeader_1x05_P2.54mm_Vertical, symbol Connector:Conn_01x05_Pin
- added J24: I Channel SMA, Connector_Coaxial:SMA_Amphenol_132289_EdgeMount, symbol Connector:Conn_Coaxial
- added J25: Q Channel SMA, Connector_Coaxial:SMA_Amphenol_132289_EdgeMount, symbol Connector:Conn_Coaxial
- added J26: IF_input, Connector_Coaxial:SMA_Amphenol_132289_EdgeMount, symbol Connector:Conn_Coaxial
- added J27: rf_test, Connector_PinHeader_2.54mm:PinHeader_1x02_P2.54mm_Vertical, symbol Connector:Conn_01x02_Pin
- added J28: I_clk_test, Connector_PinHeader_2.54mm:PinHeader_1x02_P2.54mm_Vertical, symbol Connector:Conn_01x02_Pin
- added J29: Q_clk_test, Connector_PinHeader_2.54mm:PinHeader_1x02_P2.54mm_Vertical, symbol Connector:Conn_01x02_Pin
- added J30: Rx_Q_channel, Connector_Audio:Jack_3.5mm_CUI_SJ-3523-SMT_Horizontal, symbol audiojack3:AudioJack3
- added J31: Rx_I_channel, Connector_Audio:Jack_3.5mm_CUI_SJ-3523-SMT_Horizontal, symbol audiojack3:AudioJack3
- added J32: Tx_Q_channel, Connector_Audio:Jack_3.5mm_CUI_SJ-3523-SMT_Horizontal, symbol audiojack3:AudioJack3
- added J33: Tx_I_channel, Connector_Audio:Jack_3.5mm_CUI_SJ-3523-SMT_Horizontal, symbol audiojack3:AudioJack3
- added R10, R9: 2.2k, Resistor_SMD:R_0805_2012Metric_Pad1.20x1.40mm_HandSolder, symbol Device:R_Small_US
- added R11, R12, R13, R14: 1M, Resistor_SMD:R_0805_2012Metric_Pad1.20x1.40mm_HandSolder, symbol Device:R_Small_US
- added R8: 100, Resistor_SMD:R_0805_2012Metric_Pad1.20x1.40mm_HandSolder, symbol Device:R_Small_US
- added TR2: ADT4-6T, RF_Mini-Circuits:Mini-Circuits_CD637_H5.23mm, symbol Transformer:ADT4-6T
- added U17, U18, U7, U8: NC7SVU04P5X, Package_TO_SOT_SMD:SOT-353_SC-70-5, symbol 74xGxx:NC7SVU04P5X
- added U19, U20: SN74CBT3253, Package_SO:SOIC-16_3.9x9.9mm_P1.27mm, symbol Analog_Switch:SN74CBT3253
Connections:
- new net: C28.2, R13.2, U17.2
- new net: C34.2, J33.R, U20.10 (2B1), U20.3 (1B4)
- new net: C38.2, J32.T, U20.12 (2B3), U20.5 (1B2)
- new net: C40.2, J33.T, U20.13 (2B4), U20.6 (1B1)
- new net: C27.2, TR2.3
- new net: TR2.4, U19.7 (1A), U20.7 (1A)
- new net: TR2.6, U19.9 (2A), U20.9 (2A)
- new net: C37.2, J30.T, U19.12 (2B3), U19.5 (1B2)
- new net: C24.1, J24.1 (In)
- new net: C24.2, R11.2, U7.2
- new net: C33.2, J31.R, U19.10 (2B1), U19.3 (1B4)
- new net: C39.2, J31.T, U19.13 (2B4), U19.6 (1B1)
- new net: C27.1, J26.1 (In), J27.1 (Pin_1)
- new net: C29.1, R12.1, U8.4
- new net: C29.2, R14.2, U18.2
- new net: C36.2, J32.R, U20.11 (2B2), U20.4 (1B3)
- new net: C35.2, J30.R, U19.11 (2B2), U19.4 (1B3)
- new net: C26.1, J25.1 (In)
- new net: C26.2, R12.2, U8.2
- new net: C28.1, R11.1, U7.4
- new net +3.3V: C22.1, J23.2 (Pin_2), R8.2, R9.1
- new net +5V: C31.1, C32.1, J23.1 (Pin_1), U19.16 (VCC), U20.16 (VCC)
- new net GND: C21.2, C22.2, C23.2, C25.2, C30.2, C31.2, C32.2, C33.1, C34.1, C35.1, C36.1, C37.1, C38.1, C39.1, C40.1, J23.5 (Pin_5), J24.2 (Ext), J25.2 (Ext), J26.2 (Ext), J27.2 (Pin_2), J28.2 (Pin_2), J29.2 (Pin_2), J30.S, J31.S, J32.S, J33.S, R10.1, TR2.1, U17.3 (GND), U18.3 (GND), U19.8 (GND), U20.8 (GND), U7.3 (GND), U8.3 (GND)
- new net I_square: J28.1 (Pin_1), R13.1, U17.4, U19.14 (S0), U20.14 (S0)
- new net Q_square: J29.1 (Pin_1), R14.1, U18.4, U19.2 (S1), U20.2 (S1)
- new net Rx_control: J23.4 (Pin_4), U19.1 (1~{OE}), U19.15 (2~{OE})
- new net Tx_control: J23.3 (Pin_3), U20.1 (1~{OE}), U20.15 (2~{OE})
- new net V_inverter: C21.1, C23.1, C25.1, R8.1, U17.5 (VCC), U18.5 (VCC), U7.5 (VCC), U8.5 (VCC)
- new net bias: C30.1, R10.2, R9.2, TR2.5
Other:
- note added: "Detector Bias Circuit"
- note added: "Inverter Power"
- note added: "Power Flags"
- note added: "Power and Control"
- note added: "Quadrature Clocks"
- note added: "Receive Mixer"
- note added: "Transmit Mixer"

Commit message: selected clocking scheme
Parts:
- removed C21, C22: 47u, Capacitor_SMD:C_0805_2012Metric_Pad1.18x1.45mm_HandSolder, symbol Device:C_Polarized_Small_US
- removed C23, C24, C25, C26, C27, C28, C29, C30, C31, C32: 0.1u, Capacitor_SMD:C_0805_2012Metric_Pad1.18x1.45mm_HandSolder, symbol Device:C_Small
- removed C33, C34, C35, C36, C37, C38, C39, C40: 0.068u, Capacitor_SMD:C_0805_2012Metric_Pad1.18x1.45mm_HandSolder, symbol Device:C_Small
- removed H5, H6, H7, H8: MountingHole, MountingHole:MountingHole_3.2mm_M3, symbol Mechanical:MountingHole
- removed J23: Conn_01x05_Pin, Connector_PinHeader_2.54mm:PinHeader_1x05_P2.54mm_Vertical, symbol Connector:Conn_01x05_Pin
- removed J24: I Channel SMA, Connector_Coaxial:SMA_Amphenol_132289_EdgeMount, symbol Connector:Conn_Coaxial
- removed J25: Q Channel SMA, Connector_Coaxial:SMA_Amphenol_132289_EdgeMount, symbol Connector:Conn_Coaxial
- removed J26: IF_input, Connector_Coaxial:SMA_Amphenol_132289_EdgeMount, symbol Connector:Conn_Coaxial
- removed J27: rf_test, Connector_PinHeader_2.54mm:PinHeader_1x02_P2.54mm_Vertical, symbol Connector:Conn_01x02_Pin
- removed J28: I_clk_test, Connector_PinHeader_2.54mm:PinHeader_1x02_P2.54mm_Vertical, symbol Connector:Conn_01x02_Pin
- removed J29: Q_clk_test, Connector_PinHeader_2.54mm:PinHeader_1x02_P2.54mm_Vertical, symbol Connector:Conn_01x02_Pin
- removed J30: Rx_Q_channel, Connector_Audio:Jack_3.5mm_CUI_SJ-3523-SMT_Horizontal, symbol audiojack3:AudioJack3
- removed J31: Rx_I_channel, Connector_Audio:Jack_3.5mm_CUI_SJ-3523-SMT_Horizontal, symbol audiojack3:AudioJack3
- removed J32: Tx_Q_channel, Connector_Audio:Jack_3.5mm_CUI_SJ-3523-SMT_Horizontal, symbol audiojack3:AudioJack3
- removed J33: Tx_I_channel, Connector_Audio:Jack_3.5mm_CUI_SJ-3523-SMT_Horizontal, symbol audiojack3:AudioJack3
- removed R10, R9: 2.2k, Resistor_SMD:R_0805_2012Metric_Pad1.20x1.40mm_HandSolder, symbol Device:R_Small_US
- removed R11, R12, R13, R14: 1M, Resistor_SMD:R_0805_2012Metric_Pad1.20x1.40mm_HandSolder, symbol Device:R_Small_US
- removed R8: 100, Resistor_SMD:R_0805_2012Metric_Pad1.20x1.40mm_HandSolder, symbol Device:R_Small_US
- removed TR2: ADT4-6T, RF_Mini-Circuits:Mini-Circuits_CD637_H5.23mm, symbol Transformer:ADT4-6T
- removed U17, U18, U7, U8: NC7SVU04P5X, Package_TO_SOT_SMD:SOT-353_SC-70-5, symbol 74xGxx:NC7SVU04P5X
- removed U19, U20: SN74CBT3253, Package_SO:SOIC-16_3.9x9.9mm_P1.27mm, symbol Analog_Switch:SN74CBT3253
Other:
- note removed: "Detector Bias Circuit"
- note removed: "Inverter Power"
- note removed: "Power Flags"
- note removed: "Power and Control"
- note removed: "Quadrature Clocks"
- note removed: "Receive Mixer"
- note removed: "Transmit Mixer"
