File: sdr_12p/adau1962a.kicad_sch (KiCad schematic)
At the start: 0 parts

Commit message: basic arrangement of blocks
Parts:
- added U5: ADAU1962AWBSTZ, ST_80_2_ADI, symbol ADAU1962A:ADAU1962AWBSTZ
Other:
- company: (none) -> Andy McCann KA3KAF and Doug McCann KA3KAG
- title: (none) -> Transmit DACs
Changed lines of the file:
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@@
 	(generator "eeschema")
 	(generator_version "9.0")
-	(paper "A4")
+	(paper "B")
+	(title_block
+		(title "Transmit DACs")
+		(date "2026-01-02")
+		(rev "0.0")
+		(company "Andy McCann KA3KAF and Doug McCann KA3KAG")
+	)
+	(symbol
+		(lib_id "ADAU1962A:ADAU1962AWBSTZ")
+		(at 102.87 35.56 0)
+		(unit 1)
+		(exclude_from_sim no)
+		(in_bom yes)
+		(on_board yes)
+		(dnp no)
+		(fields_autoplaced yes)
+		(property "Reference" "U5"
+			(at 140.97 25.4 0)
+			(effects
+				(font
+					(size 1.524 1.524)
+				)
+			)
+		)
+		(property "Value" "ADAU1962AWBSTZ"
+			(at 140.97 27.94 0)
+			(effects
+				(font
+					(size 1.524 1.524)
+				)
+			)
+		)
+		(property "Footprint" "ST_80_2_ADI"
+			(at 102.87 35.56 0)
+			(effects
+				(font
+					(size 1.27 1.27)
+					(italic yes)
+				)
+				(hide yes)
+			)
+		)
+		(property "Datasheet" "https://www.analog.com/media/en/technical-documentation/data-sheets/ADAU1962A.pdf"
+			(at 102.87 35.56 0)
+			(effects
+				(font
+					(size 1.27 1.27)
+					(italic yes)
+				)
+				(hide yes)
+			)
+		)
+		(property "Description" ""
+			(at 102.87 35.56 0)
+			(effects
+				(font
+					(size 1.27 1.27)
+				)
+				(hide yes)
+			)
+		)
+		(pin "48"
+		)
+		(pin "49"
+		)
+		(pin "35"
+		)
+		(pin "27"
+		)
+		(pin "29"
+		)
+		(pin "57"
+		)
+		(pin "75"
+		)
+		(pin "76"
+		)
+		(pin "74"
+		)
+		(pin "39"
+		)
+		(pin "80"
+		)
+		(pin "64"
+		)
+		(pin "8"
+		)
+		(pin "69"
+		)
+		(pin "45"
+		)
+		(pin "44"
+		)
+		(pin "43"
+		)
+		(pin "46"
+		)
+		(pin "62"
+		)
+		(pin "23"
+		)
+		(pin "51"
+		)
+		(pin "2"
+		)
+		(pin "5"
+		)
+		(pin "20"
+		)
+		(pin "52"
+		)
+		(pin "36"
+		)
+		(pin "54"
+		)
+		(pin "66"
+		)
+		(pin "50"
+		)
+		(pin "63"
+		)
+		(pin "79"
+		)
+		(pin "60"
+		)
+		(pin "37"
+		)
+		(pin "59"
+		)
+		(pin "58"
+		)
+		(pin "61"
+		)
+		(pin "1"
+		)
+		(pin "21"
+		)
+		(pin "78"
+		)
+		(pin "71"
+		)
+		(pin "38"
+		)
+		(pin "13"
+		)
+		(pin "24"
+		)
+		(pin "28"
+		)
+		(pin "70"
+		)
+		(pin "18"
+		)
+		(pin "56"
+		)
+		(pin "73"
+		)
+		(pin "6"
+		)
+		(pin "9"
+		)
+		(pin "33"
+		)
+		(pin "17"
+		)
+		(pin "25"
+		)
+		(pin "22"
+		)
+		(pin "15"
+		)
+		(pin "65"
+		)
+		(pin "7"
+		)
+		(pin "53"
+		)
+		(pin "30"
+		)
+		(pin "32"
+		)
+		(pin "19"
+		)
+		(pin "55"
+		)
+		(pin "77"
+		)
+		(pin "41"
+		)
+		(pin "16"
+		)
+		(pin "42"
+		)
+		(pin "10"
+		)
+		(pin "47"
+		)
+		(pin "26"
+		)
+		(pin "11"
+		)
+		(pin "31"
+		)
+		(pin "14"
+		)
+		(pin "40"
+		)
+		(pin "72"
+		)
+		(pin "68"
+		)
+		(pin "34"
+		)
+		(pin "67"
+		)
+		(pin "4"
+		)
+		(pin "3"
+		)
+		(pin "12"
+		)
+		(instances
+			(project ""
+				(path "/fe42ca2f-2bb8-4d5a-9e84-807788ed632f/1097e363-2947-4914-97f0-a09e0bb38c3a"
+					(reference "U5")
+					(unit 1)
+				)
+			)
+		)
+	)
 )
