File: sdr_12p/power_mgmt.kicad_sch (KiCad schematic)
At the start: 0 parts

Commit message: added rx switches
Parts:
- added C1, C3, C74, C80: 4.7u, Capacitor_SMD:C_0603_1608Metric_Pad1.08x0.95mm_HandSolder, symbol Device:C_Small
- added C10, C4, C5, C7, C73, C76, C77, C78, C79, C8, C81, C9: 2.2u, symbol Device:C_Small
- added C2, C75: 0.47u, Capacitor_SMD:C_0603_1608Metric_Pad1.08x0.95mm_HandSolder, symbol Device:C_Small
- added C34, C39: 10uF 25V, Capacitor_SMD:C_0603_1608Metric, symbol Device:C_Small
- added C35, C40: 0.1u, Capacitor_SMD:C_0603_1608Metric, symbol Device:C_Small
- added C36, C37, C38, C43, C71, C72: 47u 6.3V, Capacitor_SMD:C_0603_1608Metric, symbol Device:C_Small
- added D4, D5: B330, Diode_SMD:D_SMC, symbol Diode:B330
- added L1, L2: 3.3u 3A, Inductor_SMD:L_Abracon_ASPI-0630LR, symbol Device:L_Small
- added R1, R8: 49.9, Resistor_SMD:R_0603_1608Metric_Pad0.98x0.95mm_HandSolder, symbol Device:R_Small_US
- added R2, R4, R6, R7: ~, Resistor_SMD:R_0603_1608Metric, symbol Device:R_Small_US
- added R3, R5: 100k, Resistor_SMD:R_0603_1608Metric, symbol Device:R_Small_US
- added U36, U37: ADP2302ARDZ, Package_SO:SOIC-8-1EP_3.9x4.9mm_P1.27mm_EP2.29x3mm, symbol Regulator_Switching:ADP2302ARDZ
- added U38, U4: LT3042xMSE, Package_SO:MSOP-10-1EP_3x3mm_P0.5mm_EP1.68x1.88mm, symbol Regulator_Linear:LT3042xMSE
Connections:
- new net: R3.2, U36.4 (PGOOD)
- new net: R2.2, R4.1, U36.5 (FB)
- new net: C35.1, L2.1, U36.1 (BST)
- new net: C35.2, D4.1 (K), U36.8 (SW)
- new net: R6.2, R7.1, U37.5 (FB)
- new net: C40.2, D5.1 (K), U37.8 (SW)
- new net: C75.1, R8.1, U38.7 (SET)
- new net: C40.1, L1.1, U37.1 (BST)
- new net: R5.2, U37.4 (PGOOD)
- new net: C2.1, R1.1, U4.7 (SET)
- new net +3.6V: C43.1, C71.1, C72.1, L1.2, R6.1
- new net +5.5V: C1.1, C36.1, C37.1, C38.1, C74.1, L2.2, R2.1, U38.1 (IN), U38.2 (IN), U38.3 (EN/UV), U38.6 (PGFB), U4.1 (IN), U4.2 (IN), U4.3 (EN/UV), U4.6 (PGFB)
- new net 5V: C3.1, C80.1, U38.10 (OUT), U38.9 (OUTS), U4.10 (OUT), U4.9 (OUTS)
- new net 5V_RX_SW: C73.1, C76.1, C77.1, C78.1, C79.1, C81.1
- new net 5V_TX_SW: C10.1, C4.1, C5.1, C7.1, C8.1, C9.1
- new net GND: C1.2, C10.2, C2.2, C3.2, C34.2, C36.2, C37.2, C38.2, C39.2, C4.2, C43.2, C5.2, C7.2, C71.2, C72.2, C73.2, C74.2, C75.2, C76.2, C77.2, C78.2, C79.2, C8.2, C80.2, C81.2, C9.2, D4.2 (A), D5.2 (A), R1.2, R4.2, R7.2, R8.2, U36.7 (GND), U36.9 (PADGND), U37.7 (GND), U37.9 (PADGND), U38.11 (GND), U38.5 (ILIM), U38.8 (GND), U4.11 (GND), U4.5 (ILIM), U4.8 (GND)
- new net PWR_MAIN: C34.1, C39.1, R3.1, R5.1, U36.2 (Vin), U36.3 (EN), U37.2 (Vin), U37.3 (EN)
- no-connect marks 0 -> 2
Other:
- note added: "5V Power for Rx Switches"
- note added: "5V Power for Tx Switches"
- note added: "Place one of these near each group of 4 switches"
- note added: "R1 sets 5V output Use high quality cap for C2 such as COG"
- note added: "These passive values have not been validated"
- company: (none) -> Andy McCann KA3KAG and Doug McCann KA3KAG
- title: (none) -> Power Management
