File: sdr_12p/power_ldos.kicad_sch (KiCad schematic)
At the start: 40 parts, among them U38 LT3042xMSE, U39 LT3042xMSE, U4 LT3042xMSE, U40 LT3042xMSE, U41 LT3042xMSE, U42 LT3042xMSE, U43 LT3042xMSE, U44 LT3042xMSE

Commit message: added power mgmt
Connections:
- removed net 5V: C107.1, C116.1, C125.1, C134.1, C3.1, C80.1, C89.1, C98.1, U38.10 (OUT), U38.9 (OUTS), U39.10 (OUT), U39.9 (OUTS), U4.10 (OUT), U4.9 (OUTS), U40.10 (OUT), U40.9 (OUTS), U41.10 (OUT), U41.9 (OUTS), U42.10 (OUT), U42.9 (OUTS), U43.10 (OUT), U43.9 (OUTS), U44.10 (OUT), U44.9 (OUTS)
- new net 3.3V_ADCs: C89.1, U39.10 (OUT), U39.9 (OUTS)
- new net 3.3V_DACs: C98.1, U40.10 (OUT), U40.9 (OUTS)
- new net 3.3V_DSP: C107.1, U41.10 (OUT), U41.9 (OUTS)
- new net 3.3V_PLL: C116.1, U42.10 (OUT), U42.9 (OUTS)
- new net 3.3V_RX_CLK: C134.1, U44.10 (OUT), U44.9 (OUTS)
- new net 3.3V_TX_CLK: C125.1, U43.10 (OUT), U43.9 (OUTS)
- new net 5V_RX_Mixer: C80.1, U38.10 (OUT), U38.9 (OUTS)
- new net 5V_TX_Mixer: C3.1, U4.10 (OUT), U4.9 (OUTS)
Changed lines of the file:
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@@
 		)
 	)
-	(label "5V"
-		(at 87.63 39.37 0)
-		(effects
-			(font
-				(size 1.27 1.27)
-			)
-			(justify left bottom)
-		)
-	)
-	(label "5V"
-		(at 289.56 39.37 0)
-		(effects
-			(font
-				(size 1.27 1.27)
-			)
-			(justify left bottom)
-		)
-	)
-	(label "5V"
-		(at 392.43 156.21 0)
-		(effects
-			(font
-				(size 1.27 1.27)
-			)
-			(justify left bottom)
-		)
-	)
-	(label "5V"
-		(at 187.96 39.37 0)
-		(effects
-			(font
-				(size 1.27 1.27)
-			)
-			(justify left bottom)
-		)
-	)
-	(label "5V"
+	(hierarchical_label "3.3V_RX_CLK"
+		(shape input)
 		(at 292.1 157.48 0)
-		(effects
-			(font
-				(size 1.27 1.27)
-			)
-			(justify left bottom)
-		)
-	)
-	(label "5V"
-		(at 391.16 39.37 0)
-		(effects
-			(font
-				(size 1.27 1.27)
-			)
-			(justify left bottom)
-		)
-	)
-	(label "5V"
-		(at 187.96 160.02 0)
-		(effects
-			(font
-				(size 1.27 1.27)
-			)
-			(justify left bottom)
-		)
-	)
-	(label "5V"
-		(at 87.63 160.02 0)
-		(effects
-			(font
-				(size 1.27 1.27)
-			)
-			(justify left bottom)
-		)
-	)
-	(global_label "5.5V"
-		(shape input)
-		(at 50.8 29.21 90)
-		(fields_autoplaced yes)
 		(effects
 			(font
@@
 			(justify left)
 		)
-		(property "Intersheetrefs" "${INTERSHEET_REFS}"
-			(at 50.8 22.1124 90)
-			(effects
-				(font
-					(size 1.27 1.27)
-				)
-				(justify left)
-				(hide yes)
-			)
-		)
 	)
-	(global_label "3.6V"
+	(hierarchical_label "3.6V"
 		(shape input)
-		(at 252.73 29.21 90)
-		(fields_autoplaced yes)
+		(at 355.6 146.05 90)
 		(effects
 			(font
@@
 			(justify left)
 		)
-		(property "Intersheetrefs" "${INTERSHEET_REFS}"
-			(at 252.73 22.1124 90)
-			(effects
-				(font
-					(size 1.27 1.27)
-				)
-				(justify left)
-				(hide yes)
-			)
-		)
 	)
-	(global_label "5.5V"
+	(hierarchical_label "5V_TX_Mixer"
 		(shape input)
-		(at 151.13 29.21 90)
-		(fields_autoplaced yes)
+		(at 187.96 39.37 0)
 		(effects
 			(font
@@
 			(justify left)
 		)
-		(property "Intersheetrefs" "${INTERSHEET_REFS}"
-			(at 151.13 22.1124 90)
-			(effects
-				(font
-					(size 1.27 1.27)
-				)
-				(justify left)
-				(hide yes)
-			)
-		)
 	)
-	(global_label "3.6V"
+	(hierarchical_label "3.6V"
 		(shape input)
-		(at 355.6 146.05 90)
-		(fields_autoplaced yes)
+		(at 50.8 149.86 90)
 		(effects
 			(font
@@
 			(justify left)
 		)
-		(property "Intersheetrefs" "${INTERSHEET_REFS}"
-			(at 355.6 138.9524 90)
-			(effects
-				(font
-					(size 1.27 1.27)
-				)
-				(justify left)
-				(hide yes)
-			)
-		)
 	)
-	(global_label "3.6V"
+	(hierarchical_label "3.3V_DACs"
 		(shape input)
-		(at 255.27 147.32 90)
-		(fields_autoplaced yes)
+		(at 187.96 160.02 0)
 		(effects
 			(font
@@
 			(justify left)
 		)
-		(property "Intersheetrefs" "${INTERSHEET_REFS}"
-			(at 255.27 140.2224 90)
-			(effects
-				(font
-					(size 1.27 1.27)
-				)
-				(justify left)
-				(hide yes)
-			)
-		)
 	)
-	(global_label "3.6V"
+	(hierarchical_label "3.3V_PLL"
 		(shape input)
-		(at 151.13 149.86 90)
-		(fields_autoplaced yes)
+		(at 391.16 39.37 0)
 		(effects
 			(font
@@
 			(justify left)
 		)
-		(property "Intersheetrefs" "${INTERSHEET_REFS}"
-			(at 151.13 142.7624 90)
-			(effects
-				(font
-					(size 1.27 1.27)
-				)
-				(justify left)
-				(hide yes)
-			)
-		)
 	)
-	(global_label "3.6V"
+	(hierarchical_label "3.3V_ADCs"
 		(shape input)
-		(at 354.33 29.21 90)
-		(fields_autoplaced yes)
+		(at 87.63 160.02 0)
 		(effects
 			(font
@@
 			(justify left)
 		)
-		(property "Intersheetrefs" "${INTERSHEET_REFS}"
-			(at 354.33 22.1124 90)
-			(effects
-				(font
-					(size 1.27 1.27)
-				)
-				(justify left)
-				(hide yes)
-			)
-		)
 	)
-	(global_label "3.6V"
+	(hierarchical_label "5V_RX_Mixer"
 		(shape input)
-		(at 50.8 149.86 90)
-		(fields_autoplaced yes)
+		(at 87.63 39.37 0)
 		(effects
 			(font
@@
 			(justify left)
 		)
-		(property "Intersheetrefs" "${INTERSHEET_REFS}"
-			(at 50.8 142.7624 90)
-			(effects
-				(font
-					(size 1.27 1.27)
-				)
-				(justify left)
-				(hide yes)
+	)
+	(hierarchical_label "5.5V"
+		(shape input)
+		(at 50.8 29.21 90)
+		(effects
+			(font
+				(size 1.27 1.27)
 			)
+			(justify left)
 		)
 	)
+	(hierarchical_label "3.6V"
+		(shape input)
+		(at 255.27 147.32 90)
+		(effects
+			(font
+				(size 1.27 1.27)
+			)
+			(justify left)
+		)
+	)
+	(hierarchical_label "3.6V"
+		(shape input)
+		(at 252.73 29.21 90)
+		(effects
+			(font
+				(size 1.27 1.27)
+			)
+			(justify left)
+		)
+	)
+	(hierarchical_label "3.3V_DSP"
+		(shape input)
+		(at 289.56 39.37 0)
+		(effects
+			(font
+				(size 1.27 1.27)
+			)
+			(justify left)
+		)
+	)
+	(hierarchical_label "3.6V"
+		(shape input)
+		(at 354.33 29.21 90)
+		(effects
+			(font
+				(size 1.27 1.27)
+			)
+			(justify left)
+		)
+	)
+	(hierarchical_label "5.5V"
+		(shape input)
+		(at 151.13 29.21 90)
+		(effects
+			(font
+				(size 1.27 1.27)
+			)
+			(justify left)
+		)
+	)
+	(hierarchical_label "3.3V_TX_CLK"
+		(shape input)
+		(at 392.43 156.21 0)
+		(effects
+			(font
+				(size 1.27 1.27)
+			)
+			(justify left)
+		)
+	)
+	(hierarchical_label "3.6V"
+		(shape input)
+		(at 151.13 149.86 90)
+		(effects
+			(font
+				(size 1.27 1.27)
+			)
+			(justify left)
+		)
+	)

Commit message: fixed power ldo page
Connections:
- net 3.3V_DSP renamed 3.3V_DAP
Other:
- note added: "3.3V Power for Coarse VFO"
- note added: "3.3V Power for DAP"
- note removed: "3.3V Power for DSP"
- note removed: "3.3V Power for PLL"
Changed lines of the file:
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@@
 		)
 	)
-	(text "3.3V Power for DSP"
+	(text "3.3V Power for DAP"
 		(exclude_from_sim no)
 		(at 233.172 18.288 0)
@@
 		)
 	)
-	(text "3.3V Power for PLL"
+	(text "3.3V Power for Coarse VFO"
 		(exclude_from_sim no)
 		(at 334.772 18.288 0)
@@
 		)
 	)
-	(hierarchical_label "3.3V_DSP"
+	(hierarchical_label "3.3V_DAP"
 		(shape input)
 		(at 289.56 39.37 0)
