File: sdr_12p/power_ldos.kicad_sch (KiCad schematic)
At the start: 50 parts, among them U10 LT3042xMSE, U38 LT3042xMSE, U39 LT3042xMSE, U4 LT3042xMSE, U40 LT3042xMSE, U41 LT3042xMSE, U42 LT3042xMSE, U43 LT3042xMSE, U44 LT3042xMSE, U7 LT3042xMSE

Commit message: fixed ldos for Clocks and DAP
Parts:
- removed C101, C107, C110, C116, C119, C125, C128, C134: 4.7u, Capacitor_SMD:C_0603_1608Metric_Pad1.08x0.95mm_HandSolder, symbol Device:C_Small
- removed C102, C111, C120, C129: 0.47u, Capacitor_SMD:C_0603_1608Metric_Pad1.08x0.95mm_HandSolder, symbol Device:C_Small
- removed R11: 33.2, Resistor_SMD:R_0603_1608Metric_Pad0.98x0.95mm_HandSolder, symbol Device:R_Small_US
- removed U41, U42, U43, U44: LT3042xMSE, Package_SO:MSOP-10-1EP_3x3mm_P0.5mm_EP1.68x1.88mm, symbol Regulator_Linear:LT3042xMSE
- added C33, C47, C51: 10u, Capacitor_SMD:C_0603_1608Metric_Pad1.08x0.95mm_HandSolder, symbol Device:C_Small
- added C44, C48, C52: 0.47u, Capacitor_SMD:C_0603_1608Metric_Pad1.08x0.95mm_HandSolder, symbol Device:C_Small
- added C45, C46, C49, C50, C53, C54: 4.7u, Capacitor_SMD:C_0603_1608Metric_Pad1.08x0.95mm_HandSolder, symbol Device:C_Small
- added R18, R19, R20, R21, R22, R23: 20m, Resistor_SMD:R_0603_1608Metric_Pad0.98x0.95mm_HandSolder, symbol Device:R_Small_US
- added U21, U42, U43, U44, U49, U50: LT3045xMSE, Package_SO:MSOP-12-1EP_3x4.039mm_P0.65mm_EP1.651x2.845mm, symbol Regulator_Linear:LT3045xMSE
- R10, R9: value 33.2 -> 33.2k
- R12, R13, R14: value 33.2 -> 16.5k
Connections:
- net 3.6V: now also C33.1, C47.1, C51.1, U21.1 (IN), U21.2 (IN), U21.3 (IN), U21.4 (EN/UV), U21.7 (PGFB), U42.1 (IN), U42.2 (IN), U42.3 (IN), U42.4 (EN/UV), U42.7 (PGFB), U43.1 (IN), U43.2 (IN), U43.3 (IN), U43.4 (EN/UV), U43.7 (PGFB), U44.1 (IN), U44.2 (IN), U44.3 (IN), U44.4 (EN/UV), U44.7 (PGFB), U49.1 (IN), U49.2 (IN), U49.3 (IN), U49.4 (EN/UV), U49.7 (PGFB), U50.1 (IN), U50.2 (IN), U50.3 (IN), U50.4 (EN/UV), U50.7 (PGFB)
- net GND: now also C33.2, C44.2, C45.2, C46.2, C47.2, C48.2, C49.2, C50.2, C51.2, C52.2, C53.2, C54.2, U21.13 (GND), U21.6 (ILIM), U21.9 (GND), U42.13 (GND), U42.6 (ILIM), U42.9 (GND), U43.13 (GND), U43.6 (ILIM), U43.9 (GND), U44.13 (GND), U44.6 (ILIM), U44.9 (GND), U49.13 (GND), U49.6 (ILIM), U49.9 (GND), U50.13 (GND), U50.6 (ILIM), U50.9 (GND)
- net at R14.1: now also C52.1, U44.8 (SET), U50.8 (SET)
- net at R12.1: now also C48.1, U42.8 (SET), U49.8 (SET)
- net at R13.1: now also C44.1, U21.8 (SET), U43.8 (SET)
- net 5V_RX_Mixer renamed 5V_Mixer
- new net: C45.1, R18.1, U21.10 (OUTS), U21.11 (OUT), U21.12 (OUT)
- new net: C54.1, R23.1, U50.10 (OUTS), U50.11 (OUT), U50.12 (OUT)
- new net: C46.1, R19.1, U43.10 (OUTS), U43.11 (OUT), U43.12 (OUT)
- new net: C49.1, R20.1, U42.10 (OUTS), U42.11 (OUT), U42.12 (OUT)
- new net: C53.1, R22.1, U44.10 (OUTS), U44.11 (OUT), U44.12 (OUT)
- new net: C50.1, R21.1, U49.10 (OUTS), U49.11 (OUT), U49.12 (OUT)
- new net 3.3V_Clock_Tree: R22.2, R23.2
- new net 3.3V_VCO_FANBUF: R18.2, R19.2, R20.2, R21.2
- no-connect marks 10 -> 12
Other:
- note added: "3.3V Power for Clock Tree"
- note added: "3.3V Power for Coarse VFO and Fanout Buffer"
- note added: "5V Power for Mixer Switches"
- note removed: "3.3V Power for Coarse VFO"
- note removed: "3.3V Power for Rx Clock"
- note removed: "3.3V Power for Tx Clock"
- note removed: "5V Power for Rx Switches"
