File: sdr_12p/microcontroller.kicad_sch (KiCad schematic)
At the start: 0 parts

Commit message: added uC
Parts:
- added U1: RP2040, Package_DFN_QFN:QFN-56-1EP_7x7mm_P0.4mm_EP3.2x3.2mm, symbol MCU_RaspberryPi:RP2040
Connections:
- new net: U1.1 (IOVDD), U1.10 (IOVDD), U1.22 (IOVDD), U1.33 (IOVDD), U1.42 (IOVDD), U1.49 (IOVDD)
- new net: U1.23 (DVDD), U1.50 (DVDD)
Other:
- company: (none) -> Andy McCann KA3KAF and Doug McCann KA3KAG
- title: (none) -> Microprocessor
Changed lines of the file:
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@@
 	(generator "eeschema")
 	(generator_version "9.0")
-	(paper "A4")
+	(paper "B")
+	(title_block
+		(title "Microprocessor")
+		(date "2026-01-02")
+		(rev "0.0")
+		(company "Andy McCann KA3KAF and Doug McCann KA3KAG")
+	)
+	(symbol
+		(lib_id "MCU_RaspberryPi:RP2040")
+		(at 153.67 82.55 0)
+		(unit 1)
+		(exclude_from_sim no)
+		(in_bom yes)
+		(on_board yes)
+		(dnp no)
+		(fields_autoplaced yes)
+		(property "Reference" "U1"
+			(at 155.8133 127 0)
+			(effects
+				(font
+					(size 1.27 1.27)
+				)
+				(justify left)
+			)
+		)
+		(property "Value" "RP2040"
+			(at 155.8133 129.54 0)
+			(effects
+				(font
+					(size 1.27 1.27)
+				)
+				(justify left)
+			)
+		)
+		(property "Footprint" "Package_DFN_QFN:QFN-56-1EP_7x7mm_P0.4mm_EP3.2x3.2mm"
+			(at 153.67 82.55 0)
+			(effects
+				(font
+					(size 1.27 1.27)
+				)
+				(hide yes)
+			)
+		)
+		(property "Datasheet" "https://datasheets.raspberrypi.com/rp2040/rp2040-datasheet.pdf"
+			(at 153.67 82.55 0)
+			(effects
+				(font
+					(size 1.27 1.27)
+				)
+				(hide yes)
+			)
+		)
+		(property "Description" "A microcontroller by Raspberry Pi"
+			(at 153.67 82.55 0)
+			(effects
+				(font
+					(size 1.27 1.27)
+				)
+				(hide yes)
+			)
+		)
+		(pin "41"
+		)
+		(pin "37"
+		)
+		(pin "24"
+		)
+		(pin "27"
+		)
+		(pin "40"
+		)
+		(pin "19"
+		)
+		(pin "4"
+		)
+		(pin "30"
+		)
+		(pin "10"
+		)
+		(pin "46"
+		)
+		(pin "47"
+		)
+		(pin "51"
+		)
+		(pin "39"
+		)
+		(pin "34"
+		)
+		(pin "20"
+		)
+		(pin "17"
+		)
+		(pin "2"
+		)
+		(pin "22"
+		)
+		(pin "35"
+		)
+		(pin "31"
+		)
+		(pin "13"
+		)
+		(pin "38"
+		)
+		(pin "7"
+		)
+		(pin "9"
+		)
+		(pin "36"
+		)
+		(pin "26"
+		)
+		(pin "28"
+		)
+		(pin "48"
+		)
+		(pin "56"
+		)
+		(pin "53"
+		)
+		(pin "5"
+		)
+		(pin "55"
+		)
+		(pin "54"
+		)
+		(pin "6"
+		)
+		(pin "21"
+		)
+		(pin "42"
+		)
+		(pin "8"
+		)
+		(pin "43"
+		)
+		(pin "33"
+		)
+		(pin "44"
+		)
+		(pin "50"
+		)
+		(pin "12"
+		)
+		(pin "1"
+		)
+		(pin "23"
+		)
+		(pin "16"
+		)
+		(pin "29"
+		)
+		(pin "18"
+		)
+		(pin "11"
+		)
+		(pin "49"
+		)
+		(pin "52"
+		)
+		(pin "25"
+		)
+		(pin "15"
+		)
+		(pin "3"
+		)
+		(pin "32"
+		)
+		(pin "14"
+		)
+		(pin "57"
+		)
+		(pin "45"
+		)
+		(instances
+			(project ""
+				(path "/fe42ca2f-2bb8-4d5a-9e84-807788ed632f/27cecad5-c0fc-4afc-95d0-cabdd6a56668"
+					(reference "U1")
+					(unit 1)
+				)
+			)
+		)
+	)
 )
