File: sdr_16p/power_ldos.kicad_sch (KiCad schematic)
At the start: 40 parts, among them U38 LT3042xMSE, U39 LT3042xMSE, U4 LT3042xMSE, U40 LT3042xMSE, U41 LT3042xMSE, U42 LT3042xMSE, U43 LT3042xMSE, U44 LT3042xMSE

Commit message: updated to 16 channel SE
Parts:
- added C118, C4, C41, C7: 4.7u, Capacitor_SMD:C_0603_1608Metric_Pad1.08x0.95mm_HandSolder, symbol Device:C_Small
- added C42, C5: 0.47u, Capacitor_SMD:C_0603_1608Metric_Pad1.08x0.95mm_HandSolder, symbol Device:C_Small
- added R16, R17: 49.9, Resistor_SMD:R_0603_1608Metric_Pad0.98x0.95mm_HandSolder, symbol Device:R_Small_US
- added U10, U7: LT3042xMSE, Package_SO:MSOP-10-1EP_3x3mm_P0.5mm_EP1.68x1.88mm, symbol Regulator_Linear:LT3042xMSE
Connections:
- net 3.6V: now also C41.1, U10.1 (IN), U10.2 (IN), U10.3 (EN/UV), U10.6 (PGFB)
- net 5.5V: now also C4.1, U7.1 (IN), U7.2 (IN), U7.3 (EN/UV), U7.6 (PGFB)
- net GND: now also C118.2, C4.2, C41.2, C42.2, C5.2, C7.2, R16.2, R17.2, U10.11 (GND), U10.5 (ILIM), U10.8 (GND), U7.11 (GND), U7.5 (ILIM), U7.8 (GND)
- new net: C42.1, R16.1, U10.7 (SET)
- new net: C5.1, R17.1, U7.7 (SET)
- new net 5V_RX_OPAMPS: C118.1, U10.10 (OUT), U10.9 (OUTS)
- new net 5V_TX_OPAMPS: C7.1, U7.10 (OUT), U7.9 (OUTS)
- no-connect marks 8 -> 10
Other:
- note added: "5V Power for RX op amps"
- note added: "5V Power for TX Op amps"
- note added: "Resistor sets 5V output Use high quality cap such as COG"
- note removed: "R1 sets 5V output Use high quality cap for C2 such as COG"
- moved on the sheet: C119, C120, C125, C128, C129, C134, C83, C84, C89, C92, C93, C98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
