File: sdr_16p/power_switching_reg.kicad_sch (KiCad schematic)
At the start: 22 parts, among them U36 ADP2302ARDZ, U37 ADP2302ARDZ

Commit message: back to 16 phases
Parts:
- removed U36, U37: ADP2302ARDZ, Package_SO:SOIC-8-1EP_3.9x4.9mm_P1.27mm_EP2.29x3mm, symbol Regulator_Switching:ADP2302ARDZ
- added U36, U37: ADP2303ARDZ, Package_SO:SOIC-8-1EP_3.9x4.9mm_P1.27mm_EP2.29x3mm, symbol Regulator_Switching:ADP2303ARDZ
Connections:
- net GND: now also U36.7 (GND), U36.9 (PADGND), U37.7 (GND), U37.9 (PADGND)
- net MAIN: now also U36.2 (Vin), U36.3 (EN), U37.2 (Vin), U37.3 (EN)
- net at R3.2: now also U36.4 (PGOOD)
- net at R2.2, R4.1: now also U36.5 (FB)
- net at C35.1, L2.1: now also U36.1 (BST)
- net at C35.2, D4.1 (K): now also U36.8 (SW)
- net at R6.2, R7.1: now also U37.5 (FB)
- net at C40.2, D5.1 (K): now also U37.8 (SW)
- net at C40.1, L1.1: now also U37.1 (BST)
- net at R5.2: now also U37.4 (PGOOD)
Other:
- note added: "These passive values all need to be properly calculated using the datasheet. The target voltages are 5.5V and 3.6V"
- note removed: "These passive values have not been validated"
- moved on the sheet: C34, C35, C36, C37, C38, C39, C40, C43, C71, C72, D4, D5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
