File: sdr_16p/audio_subsystem.kicad_sch (KiCad schematic)
At the start: 0 parts

Commit message: added audio codec
Parts:
- added C62, C63, C65, C66, C68, C70: 10u, Capacitor_SMD:C_0805_2012Metric_Pad1.18x1.45mm_HandSolder, symbol Device:C_Polarized_Small_US
- added C64, C67, C69, C77, C78: 0.1u, Capacitor_SMD:C_0805_2012Metric_Pad1.18x1.45mm_HandSolder, symbol Device:C_Small
- added C79: 9.1p, Capacitor_SMD:C_0805_2012Metric_Pad1.18x1.45mm_HandSolder, symbol Device:C_Small
- added C81, C82, C85, C86: 10u, Capacitor_SMD:C_0805_2012Metric_Pad1.18x1.45mm_HandSolder, symbol Device:C_Small
- added J3: AudioJack3, Connector_Audio:Jack_3.5mm_CUI_SJ-3523-SMT_Horizontal, symbol Connector:AudioJack3
- added L3: 1.2n, Inductor_SMD:L_0805_2012Metric_Pad1.15x1.40mm_HandSolder, symbol Device:L_Small
- added R25: 49.9, Resistor_SMD:R_0805_2012Metric_Pad1.20x1.40mm_HandSolder, symbol Device:R_Small_US
- added U20: ADAU1761BCPZ, Package_DFN_QFN:QFN-32-1EP_5x5mm_P0.5mm_EP3.45x3.45mm, symbol ADAU1761:ADAU1761BCPZ
- added X1: ASE-12.288MHz, Oscillator:Oscillator_SMD_Abracon_ASE-4Pin_3.2x2.5mm, symbol Oscillator:ASE-xxxMHz
Connections:
- new net: C81.2, U20.10 (LINP)
- new net: C85.2, U20.12 (RINP)
- new net: J3.R, U20.19 (RHP)
- new net: J3.T, U20.20 (LHP)
- new net: C68.2, C69.2
- new net: C86.2, U20.13 (RINN)
- new net: C79.1, L3.2
- new net: R25.1, X1.3 (OUT)
- new net: C82.2, U20.11 (LINN)
- new net +3.3V: C65.1, C66.1, C67.2, C68.1, C69.1, C70.1, C77.1, C78.1, L3.1, U20.1 (IOVDD), U20.23 (AVDD), U20.30 (ADDR1/CDATA), U20.8 (AVDD), X1.1 (EN), X1.4 (Vdd)
- new net ADC_SDATA0: U20.26 (ADC_SDATA/_GPIO1)
- new net BCLK0: U20.28 (BCLK/GPIO2)
- new net CM0: U20.7 (CM)
- new net DAC_SDATA0: U20.27 (DAC_SDATA/_GPIO0)
- new net DVDDOUT0: C63.2, C64.2, U20.24 (DVDDOUT)
- new net GND: C63.1, C64.1, C66.2, C67.1, C70.2, C77.2, C78.2, C79.2, J3.S, U20.22 (AGND), U20.25 (DGND), U20.3 (ADDR0/CLATCH), U20.33 (EP), U20.9 (AGND), X1.2 (GND)
- new net LAUX0: U20.6 (LAUX)
- new net LINN0: C82.1
- new net LINP0: C81.1
- new net LOUTN0: U20.17 (LOUTN)
- new net LOUTP0: U20.18 (LOUTP)
- new net LRCLK0: U20.29 (LRCLK/GPIO3)
- new net MCLK0: R25.2, U20.2 (MCLK)
- new net MICBIAS0: U20.5 (MICBIAS)
- new net MONOOUT0: U20.21 (MONOOUT)
- new net RAUX0: U20.14 (RAUX)
- new net RINN0: C86.1
- new net RINP0: C85.1
- new net ROUTN0: U20.16 (ROUTN)
- new net ROUTP0: U20.15 (ROUTP)
- new net SCL0: U20.32 (SCL/CCLK)
- new net SDA0: U20.31 (SDA/COUT)
- no-connect marks 0 -> 1
Other:
- note added: "Audio Codec"
- note added: "Power Supply Filtering for Codec"
