File: nzif/crosspoint.kicad_sch (KiCad schematic)
At the start: 8 parts, among them U1 SN74CBT16212CDL

Commit message: fixed file names
Parts:
- gave numbers to parts that had none: 1
Changed lines of the file:
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@@
 		(dnp no)
 		(fields_autoplaced yes)
-		(property "Reference" "#PWR09"
+		(property "Reference" "#PWR?"
 			(at 96.52 219.71 0)
 			(effects
@@
 				)
 			)
+			(project "nzif"
+				(path "/fe42ca2f-2bb8-4d5a-9e84-807788ed632f/173d5eca-f61f-4af5-84ba-0d581841d6d2"
+					(reference "#PWR?")
+					(unit 1)
+				)
+			)
 		)
 	)
@@
 		(on_board yes)
 		(dnp no)
-		(property "Reference" "R1"
+		(property "Reference" "R?"
 			(at 128.27 68.58 90)
 			(effects
@@
 				)
 			)
+			(project "nzif"
+				(path "/fe42ca2f-2bb8-4d5a-9e84-807788ed632f/173d5eca-f61f-4af5-84ba-0d581841d6d2"
+					(reference "R?")
+					(unit 1)
+				)
+			)
 		)
 	)
@@
 		(dnp no)
 		(fields_autoplaced yes)
-		(property "Reference" "U1"
+		(property "Reference" "U?"
 			(at 181.61 152.4 0)
 			(effects
@@
 				)
 			)
+			(project "nzif"
+				(path "/fe42ca2f-2bb8-4d5a-9e84-807788ed632f/173d5eca-f61f-4af5-84ba-0d581841d6d2"
+					(reference "U?")
+					(unit 1)
+				)
+			)
 		)
 	)
@@
 		(dnp no)
 		(fields_autoplaced yes)
-		(property "Reference" "U?"
+		(property "Reference" "U47"
 			(at 181.61 64.77 0)
 			(effects
@@
 		(dnp no)
 		(fields_autoplaced yes)
-		(property "Reference" "FB1"
+		(property "Reference" "FB?"
 			(at 97.79 106.6418 0)
 			(effects
@@
 				)
 			)
+			(project "nzif"
+				(path "/fe42ca2f-2bb8-4d5a-9e84-807788ed632f/173d5eca-f61f-4af5-84ba-0d581841d6d2"
+					(reference "FB?")
+					(unit 1)
+				)
+			)
 		)
 	)
@@
 		(dnp no)
 		(fields_autoplaced yes)
-		(property "Reference" "#PWR05"
+		(property "Reference" "#PWR?"
 			(at 119.38 74.93 0)
 			(effects
@@
 				)
 			)
+			(project "nzif"
+				(path "/fe42ca2f-2bb8-4d5a-9e84-807788ed632f/173d5eca-f61f-4af5-84ba-0d581841d6d2"
+					(reference "#PWR?")
+					(unit 1)
+				)
+			)
 		)
 	)
@@
 		(dnp no)
 		(fields_autoplaced yes)
-		(property "Reference" "#PWR07"
+		(property "Reference" "#PWR?"
 			(at 83.82 129.54 0)
 			(effects
@@
 				)
 			)
+			(project "nzif"
+				(path "/fe42ca2f-2bb8-4d5a-9e84-807788ed632f/173d5eca-f61f-4af5-84ba-0d581841d6d2"
+					(reference "#PWR?")
+					(unit 1)
+				)
+			)
 		)
 	)
@@
 		(dnp no)
 		(fields_autoplaced yes)
-		(property "Reference" "#PWR08"
+		(property "Reference" "#PWR?"
 			(at 97.79 129.54 0)
 			(effects
@@
 				)
 			)
+			(project "nzif"
+				(path "/fe42ca2f-2bb8-4d5a-9e84-807788ed632f/173d5eca-f61f-4af5-84ba-0d581841d6d2"
+					(reference "#PWR?")
+					(unit 1)
+				)
+			)
 		)
 	)
@@
 		(dnp no)
 		(fields_autoplaced yes)
-		(property "Reference" "C2"
+		(property "Reference" "C?"
 			(at 100.33 119.5069 0)
 			(effects
@@
 				)
 			)
+			(project "nzif"
+				(path "/fe42ca2f-2bb8-4d5a-9e84-807788ed632f/173d5eca-f61f-4af5-84ba-0d581841d6d2"
+					(reference "C?")
+					(unit 1)
+				)
+			)
 		)
 	)
@@
 		(dnp no)
 		(fields_autoplaced yes)
-		(property "Reference" "C3"
+		(property "Reference" "C?"
 			(at 99.06 209.6769 0)
 			(effects
@@
 				)
 			)
+			(project "nzif"
+				(path "/fe42ca2f-2bb8-4d5a-9e84-807788ed632f/173d5eca-f61f-4af5-84ba-0d581841d6d2"
+					(reference "C?")
+					(unit 1)
+				)
+			)
 		)
 	)
@@
 		(dnp no)
 		(fields_autoplaced yes)
-		(property "Reference" "C1"
+		(property "Reference" "C?"
 			(at 86.36 119.5069 0)
 			(effects
@@
 				)
 			)
+			(project "nzif"
+				(path "/fe42ca2f-2bb8-4d5a-9e84-807788ed632f/173d5eca-f61f-4af5-84ba-0d581841d6d2"
+					(reference "C?")
+					(unit 1)
+				)
+			)
 		)
 	)
@@
 		(dnp no)
 		(fields_autoplaced yes)
-		(property "Reference" "#PWR06"
+		(property "Reference" "#PWR?"
 			(at 252.73 74.93 0)
 			(effects
@@
 				)
 			)
+			(project "nzif"
+				(path "/fe42ca2f-2bb8-4d5a-9e84-807788ed632f/173d5eca-f61f-4af5-84ba-0d581841d6d2"
+					(reference "#PWR?")
+					(unit 1)
+				)
+			)
 		)
 	)
@@
 		(dnp no)
 		(fields_autoplaced yes)
-		(property "Reference" "#PWR01"
+		(property "Reference" "#PWR?"
 			(at 146.05 153.67 0)
 			(effects
@@
 				)
 			)
+			(project "nzif"
+				(path "/fe42ca2f-2bb8-4d5a-9e84-807788ed632f/173d5eca-f61f-4af5-84ba-0d581841d6d2"
+					(reference "#PWR?")
+					(unit 1)
+				)
+			)
 		)
 	)
@@
 		(dnp no)
 		(fields_autoplaced yes)
-		(property "Reference" "#PWR04"
+		(property "Reference" "#PWR?"
 			(at 219.71 248.92 0)
 			(effects
@@
 				)
 			)
+			(project "nzif"
+				(path "/fe42ca2f-2bb8-4d5a-9e84-807788ed632f/173d5eca-f61f-4af5-84ba-0d581841d6d2"
+					(reference "#PWR?")
+					(unit 1)
+				)
+			)
 		)
 	)
@@
 		(dnp no)
 		(fields_autoplaced yes)
-		(property "Reference" "#PWR03"
+		(property "Reference" "#PWR?"
 			(at 146.05 250.19 0)
 			(effects
@@
 				)
 			)
+			(project "nzif"
+				(path "/fe42ca2f-2bb8-4d5a-9e84-807788ed632f/173d5eca-f61f-4af5-84ba-0d581841d6d2"
+					(reference "#PWR?")
+					(unit 1)
+				)
+			)
 		)
 	)
@@
 		(dnp no)
 		(fields_autoplaced yes)
-		(property "Reference" "R2"
+		(property "Reference" "R?"
 			(at 243.84 68.58 90)
 			(effects
@@
 				)
 			)
+			(project "nzif"
+				(path "/fe42ca2f-2bb8-4d5a-9e84-807788ed632f/173d5eca-f61f-4af5-84ba-0d581841d6d2"
+					(reference "R?")
+					(unit 1)
+				)
+			)
 		)
 	)
@@
 		(dnp no)
 		(fields_autoplaced yes)
-		(property "Reference" "#PWR02"
+		(property "Reference" "#PWR?"
 			(at 219.71 153.67 0)
 			(effects
@@
 					(unit 1)
 				)
+			)
+			(project "nzif"
+				(path "/fe42ca2f-2bb8-4d5a-9e84-807788ed632f/173d5eca-f61f-4af5-84ba-0d581841d6d2"
+					(reference "#PWR?")
+					(unit 1)
+				)
