File: nzif/nzif.kicad_sch (KiCad schematic)
At the start: 9 parts, among them J1 Rx, J10 ADAU1467_GPIOS, J11 ADAU1467_AUX_ADCS, J4 6V, J6 Microcontroller, J7 USBi, J8 I2S2, J9 I2S1

Commit message: fixed file names
Other:
- sheet DAP renamed DSP
- sheet DSP: file dap.kicad_sch -> dsp.kicad_sch
Changed lines of the file:
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@@
 		)
 		(instances
-			(project "sdr_16p"
+			(project "nzif"
 				(path "/fe42ca2f-2bb8-4d5a-9e84-807788ed632f"
 					(page "3")
@@
 		)
 		(instances
-			(project "sdr_16p"
+			(project "nzif"
 				(path "/fe42ca2f-2bb8-4d5a-9e84-807788ed632f"
 					(page "13")
@@
 		)
 		(instances
-			(project "sdr_16p"
+			(project "nzif"
 				(path "/fe42ca2f-2bb8-4d5a-9e84-807788ed632f"
 					(page "10")
@@
 		)
 		(instances
-			(project "sdr_16p"
+			(project "nzif"
 				(path "/fe42ca2f-2bb8-4d5a-9e84-807788ed632f"
 					(page "11")
@@
 		)
 		(instances
-			(project "sdr_16p"
+			(project "nzif"
 				(path "/fe42ca2f-2bb8-4d5a-9e84-807788ed632f"
 					(page "7")
@@
 		)
 		(instances
-			(project "sdr_16p"
+			(project "nzif"
 				(path "/fe42ca2f-2bb8-4d5a-9e84-807788ed632f"
 					(page "8")
@@
 		)
 		(instances
-			(project "sdr_16p"
+			(project "nzif"
 				(path "/fe42ca2f-2bb8-4d5a-9e84-807788ed632f"
 					(page "15")
@@
 		)
 		(instances
-			(project "sdr_16p"
+			(project "nzif"
 				(path "/fe42ca2f-2bb8-4d5a-9e84-807788ed632f"
 					(page "2")
@@
 		)
 		(instances
-			(project "sdr_16p"
+			(project "nzif"
 				(path "/fe42ca2f-2bb8-4d5a-9e84-807788ed632f"
 					(page "9")
@@
 		)
 		(instances
-			(project "sdr_16p"
+			(project "nzif"
 				(path "/fe42ca2f-2bb8-4d5a-9e84-807788ed632f"
 					(page "5")
@@
 		)
 		(instances
-			(project "sdr_16p"
+			(project "nzif"
 				(path "/fe42ca2f-2bb8-4d5a-9e84-807788ed632f"
 					(page "12")
@@
 		)
 		(instances
-			(project "sdr_16p"
+			(project "nzif"
 				(path "/fe42ca2f-2bb8-4d5a-9e84-807788ed632f"
 					(page "11")
@@
 		)
 		(instances
-			(project "sdr_16p"
+			(project "nzif"
 				(path "/fe42ca2f-2bb8-4d5a-9e84-807788ed632f"
 					(page "14")
@@
 			(color 0 0 0 0.0000)
 		)
-		(property "Sheetname" "DAP"
+		(property "Sheetname" "DSP"
 			(at 259.08 56.4384 0)
 			(effects
@@
 			)
 		)
-		(property "Sheetfile" "dap.kicad_sch"
+		(property "Sheetfile" "dsp.kicad_sch"
 			(at 259.08 170.7646 0)
 			(effects
@@
 		)
 		(instances
-			(project "sdr_16p"
+			(project "nzif"
 				(path "/fe42ca2f-2bb8-4d5a-9e84-807788ed632f"
 					(page "4")

Commit message: updated mixer block
Other:
- sheet Mixers renamed Rx_mixer
- sheet Rx_mixer: file mixers.kicad_sch -> rx_mixer.kicad_sch
Changed lines of the file:
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@@
 			(color 0 0 0 0.0000)
 		)
-		(property "Sheetname" "Mixers"
+		(property "Sheetname" "Rx_mixer"
 			(at 40.64 78.0284 0)
 			(effects
@@
 			)
 		)
-		(property "Sheetfile" "mixers.kicad_sch"
+		(property "Sheetfile" "rx_mixer.kicad_sch"
 			(at 40.64 113.6146 0)
 			(effects

Commit message: crosspoint removed
Other:
- removed sheet Crosspoint
- moved on the sheet: J1, TR1

Commit message: removed pullups from ADC page and added reminder note to top level
Other:
- note added: "Add pullup resistors to I2C clock and data lines"
Changed lines of the file:
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@@
 		(company "Andy McCann KA3KAF and Doug McCann KA3KAG")
+	)
+	(text "Add pullup resistors to I2C clock and data lines"
+		(exclude_from_sim no)
+		(at 223.52 35.052 0)
+		(effects
+			(font
+				(size 1.27 1.27)
+			)
+		)
 	)
 	(junction

Commit message: removed audio fanout buffer
Other:
- removed sheet Audio_Clock_Fanout
Changed lines of the file:
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@@
-	)
-	(sheet
-		(at 257.175 19.05)
-		(size 48.895 31.115)
-		(exclude_from_sim no)
-		(in_bom yes)
-		(on_board yes)
-		(dnp no)
-		(fields_autoplaced yes)
-		(stroke
-			(width 0.1524)
-			(type solid)
-		)
-		(fill
-			(color 0 0 0 0.0000)
-		)
-		(property "Sheetname" "Audio_Clock_Fanout"
-			(at 257.175 18.3384 0)
-			(effects
-				(font
-					(size 1.27 1.27)
-				)
-				(justify left bottom)
-			)
-		)
-		(property "Sheetfile" "audio_clock_fanout.kicad_sch"
-			(at 257.175 50.7496 0)
-			(effects
-				(font
-					(size 1.27 1.27)
-				)
-				(justify left top)
-			)
-		)
-		(instances
-			(project "nzif"
-				(path "/fe42ca2f-2bb8-4d5a-9e84-807788ed632f"
-					(page "14")
-				)
-			)
-		)
 	)
 	(sheet

Commit message: fixed the transformer selection
Parts:
- removed TR1: ADT9-1T, RF_Mini-Circuits:Mini-Circuits_CD542_H2.84mm, symbol Transformer:ADT9-1T
- added TR201: ADT2-1T, RF_Mini-Circuits:Mini-Circuits_CD542_H2.84mm, symbol Transformer:ADT2-1T
Changed lines of the file:
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@@
+	)
+	(symbol
+		(lib_id "Transformer:ADT2-1T")
+		(at 41.91 38.1 0)
+		(unit 1)
+		(exclude_from_sim no)
+		(in_bom yes)
+		(on_board yes)
+		(dnp no)
+		(fields_autoplaced yes)
+		(property "Reference" "TR201"
+			(at 41.91 27.94 0)
+			(effects
+				(font
+					(size 1.27 1.27)
+				)
+			)
+		)
+		(property "Value" "ADT2-1T"
+			(at 41.91 30.48 0)
+			(effects
+				(font
+					(size 1.27 1.27)
+				)
+			)
+		)
+		(property "Footprint" "RF_Mini-Circuits:Mini-Circuits_CD542_H2.84mm"
+			(at 41.91 46.99 0)
+			(effects
+				(font
+					(size 1.27 1.27)
+				)
+				(hide yes)
+			)
+		)
+		(property "Datasheet" "https://www.minicircuits.com/pdfs/ADT2-1T+.pdf"
+			(at 41.91 38.1 0)
+			(effects
+				(font
+					(size 1.27 1.27)
+				)
+				(hide yes)
+			)
+		)
+		(property "Description" "0.40-450MHz 1:2 RF Transformer, Unbalanced to Balanced Center Tap, CD542"
+			(at 41.91 38.1 0)
+			(effects
+				(font
+					(size 1.27 1.27)
+				)
+				(hide yes)
+			)
+		)
+		(pin "2"
+		)
+		(pin "6"
+		)
+		(pin "5"
+		)
+		(pin "4"
+		)
+		(pin "3"
+		)
+		(pin "1"
+		)
+		(instances
+			(project ""
+				(path "/fe42ca2f-2bb8-4d5a-9e84-807788ed632f"
+					(reference "TR201")
+					(unit 1)
+				)
+			)
+		)
 	)
 	(symbol
@@
 					(unit 1)
 				)
-			)
-		)
-	)
-	(symbol
-		(lib_id "Transformer:ADT9-1T")
-		(at 40.64 38.1 0)
-		(unit 1)
-		(exclude_from_sim no)
-		(in_bom yes)
-		(on_board yes)
-		(dnp no)
-		(fields_autoplaced yes)
-		(property "Reference" "TR1"
-			(at 40.64 27.94 0)
-			(effects
-				(font
-					(size 1.27 1.27)
-				)
-			)
-		)
-		(property "Value" "ADT9-1T"
-			(at 40.64 30.48 0)
-			(effects
-				(font
-					(size 1.27 1.27)
-				)
-			)
-		)
-		(property "Footprint" "RF_Mini-Circuits:Mini-Circuits_CD542_H2.84mm"
-			(at 40.64 46.99 0)
-			(effects
-				(font
-					(size 1.27 1.27)
-				)
-				(hide yes)
-			)
-		)
-		(property "Datasheet" "https://www.minicircuits.com/pdfs/ADT9-1T+.pdf"
-			(at 40.64 38.1 0)
-			(effects
-				(font
-					(size 1.27 1.27)
-				)
-				(hide yes)
-			)
-		)
-		(property "Description" "1-250MHz 1:9 RF Transformer, Unbalanced to Balanced Center Tap, CD542"
-			(at 40.64 38.1 0)
-			(effects
-				(font
-					(size 1.27 1.27)
-				)
-				(hide yes)
-			)
-		)
-		(pin "6"
-		)
-		(pin "4"
-		)
-		(pin "3"
-		)
-		(pin "5"
-		)
-		(pin "1"
-		)
-		(pin "2"
-		)
-		(instances
-			(project ""
-				(path "/fe42ca2f-2bb8-4d5a-9e84-807788ed632f"
-					(reference "TR1")
-					(unit 1)
-				)

Commit message: Further connections to DSP (Ref #3 #25)
Parts:
- added D?: Green LED, symbol Device:LED_Small_Filled
- added J?: Conn_02x05_Odd_Even, symbol Connector_Generic:Conn_02x05_Odd_Even
- added R218, R219: 33, symbol Device:R_Small_US
- added R218: 1k, symbol Device:R_Small_US
Connections:
- net GND: now also D?.1 (K), J?.10 (Pin_10), J?.5 (Pin_5), J?.7 (Pin_7), J?.8 (Pin_8), J?.9 (Pin_9)
- new net: J?.1 (Pin_1), R218.1
- new net: J?.3 (Pin_3), R219.1
- new net: D?.2 (A), R218.2
- new net +5V: J?.4 (Pin_4), R218.1
- new net IOVDD: R218.2, R219.2
- new net USB_~{RESET}: J?.6 (Pin_6)
- no-connect marks 0 -> 1
Other:
- note added: "USB Reset SPI 10 Pin Connector"

Commit message: removed coarse VFO from plan
Other:
- removed sheet Coarse_VFO
Changed lines of the file:
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@@
-	)
-	(sheet
-		(at 200.66 73.025)
-		(size 41.91 36.83)
-		(exclude_from_sim no)
-		(in_bom yes)
-		(on_board yes)
-		(dnp no)
-		(fields_autoplaced yes)
-		(stroke
-			(width 0.1524)
-			(type solid)
-		)
-		(fill
-			(color 0 0 0 0.0000)
-		)
-		(property "Sheetname" "Coarse_VFO"
-			(at 200.66 72.3134 0)
-			(effects
-				(font
-					(size 1.27 1.27)
-				)
-				(justify left bottom)
-			)
-		)
-		(property "Sheetfile" "coarse_vfo.kicad_sch"
-			(at 200.66 110.4396 0)
-			(effects
-				(font
-					(size 1.27 1.27)
-				)
-				(justify left top)
-			)
-		)
-		(instances
-			(project "nzif"
-				(path "/fe42ca2f-2bb8-4d5a-9e84-807788ed632f"
-					(page "8")
-				)
-			)
-		)
 	)
 	(sheet
