File: nzif/adcs.kicad_sch (KiCad schematic)
At the start: 18 parts

Commit message: changed Rx mixer from 8 phase to classic tayloe
Parts:
- gave numbers to parts that had none: 14
Changed lines of the file:
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@@
 		(dnp no)
 		(fields_autoplaced yes)
-		(property "Reference" "C?"
+		(property "Reference" "C209"
 			(at 107.95 116.8462 0)
 			(effects
@@
 		(dnp no)
 		(fields_autoplaced yes)
-		(property "Reference" "#PWR?"
+		(property "Reference" "#PWR0209"
 			(at 246.38 135.89 0)
 			(effects
@@
 		(dnp no)
 		(fields_autoplaced yes)
-		(property "Reference" "C2"
+		(property "Reference" "C?"
 			(at 243.84 90.1762 0)
 			(effects
@@
 				)
 			)
+			(project "nzif"
+				(path "/fe42ca2f-2bb8-4d5a-9e84-807788ed632f/d1b276aa-cc76-4829-b01b-98095216e3ce"
+					(reference "C?")
+					(unit 1)
+				)
+			)
 		)
 	)
@@
 		(dnp no)
 		(fields_autoplaced yes)
-		(property "Reference" "#PWR?"
+		(property "Reference" "#PWR0207"
 			(at 246.38 138.43 0)
 			(effects
@@
 		(dnp no)
 		(fields_autoplaced yes)
-		(property "Reference" "#PWR?"
+		(property "Reference" "#PWR0203"
 			(at 218.44 165.1 0)
 			(effects
@@
 		(dnp yes)
 		(fields_autoplaced yes)
-		(property "Reference" "C?"
+		(property "Reference" "C204"
 			(at 195.58 160.0135 0)
 			(effects
@@
 		(dnp no)
 		(fields_autoplaced yes)
-		(property "Reference" "#PWR?"
+		(property "Reference" "#PWR0205"
 			(at 240.03 173.99 0)
 			(effects
@@
 		(on_board yes)
 		(dnp no)
-		(property "Reference" "U?"
+		(property "Reference" "U201"
 			(at 133.604 113.792 0)
 			(effects
@@
 		(dnp no)
 		(fields_autoplaced yes)
-		(property "Reference" "#PWR?"
+		(property "Reference" "#PWR0204"
 			(at 226.06 100.33 0)
 			(effects
@@
 		(dnp no)
 		(fields_autoplaced yes)
-		(property "Reference" "C?"
+		(property "Reference" "C207"
 			(at 233.68 165.0937 90)
 			(effects
@@
 		(dnp no)
 		(fields_autoplaced yes)
-		(property "Reference" "#PWR?"
+		(property "Reference" "#PWR0202"
 			(at 248.92 100.33 0)
 			(effects
@@
 		(dnp yes)
 		(fields_autoplaced yes)
-		(property "Reference" "R?"
+		(property "Reference" "R201"
 			(at 195.58 170.1799 0)
 			(effects
@@
 		(dnp no)
 		(fields_autoplaced yes)
-		(property "Reference" "#PWR?"
+		(property "Reference" "#PWR0259"
 			(at 241.3 100.33 0)
 			(effects
@@
 		(dnp no)
 		(fields_autoplaced yes)
-		(property "Reference" "C?"
+		(property "Reference" "C201"
 			(at 176.53 149.8662 0)
 			(effects
@@
 		(on_board yes)
 		(dnp yes)
-		(property "Reference" "C?"
+		(property "Reference" "C203"
 			(at 185.42 165.0935 0)
 			(effects
@@
 		(dnp no)
 		(fields_autoplaced yes)
-		(property "Reference" "C?"
+		(property "Reference" "C210"
 			(at 97.79 116.8462 0)
 			(effects
@@
 		(dnp no)
 		(fields_autoplaced yes)
-		(property "Reference" "C3"
+		(property "Reference" "C?"
 			(at 251.46 90.1762 0)
 			(effects
@@
 				)
 			)
+			(project "nzif"
+				(path "/fe42ca2f-2bb8-4d5a-9e84-807788ed632f/d1b276aa-cc76-4829-b01b-98095216e3ce"
+					(reference "C?")
+					(unit 1)
+				)
+			)
 		)
 	)
@@
 		(dnp no)
 		(fields_autoplaced yes)
-		(property "Reference" "R?"
+		(property "Reference" "R208"
 			(at 266.7 139.7 90)
 			(effects
@@
 		(dnp no)
 		(fields_autoplaced yes)
-		(property "Reference" "R?"
+		(property "Reference" "R202"
 			(at 259.08 163.8299 0)
 			(effects
@@
 		(dnp no)
 		(fields_autoplaced yes)
-		(property "Reference" "C4"
+		(property "Reference" "C?"
 			(at 210.82 90.1762 0)
 			(effects
@@
 				)
 			)
+			(project "nzif"
+				(path "/fe42ca2f-2bb8-4d5a-9e84-807788ed632f/d1b276aa-cc76-4829-b01b-98095216e3ce"
+					(reference "C?")
+					(unit 1)
+				)
+			)
 		)
 	)
@@
 		(dnp no)
 		(fields_autoplaced yes)
-		(property "Reference" "C?"
+		(property "Reference" "C208"
 			(at 248.92 165.0937 90)
 			(effects
@@
 		(dnp no)
 		(fields_autoplaced yes)
-		(property "Reference" "#PWR?"
+		(property "Reference" "#PWR0208"
 			(at 245.11 173.99 0)
 			(effects
@@
 		(dnp no)
 		(fields_autoplaced yes)
-		(property "Reference" "#PWR?"
+		(property "Reference" "#PWR0258"
 			(at 256.54 173.99 0)
 			(effects
@@
 		(dnp no)
 		(fields_autoplaced yes)
-		(property "Reference" "#PWR?"
+		(property "Reference" "#PWR0214"
 			(at 95.25 127 0)
 			(effects
@@
 		(dnp no)
 		(fields_autoplaced yes)
-		(property "Reference" "C?"
+		(property "Reference" "C205"
 			(at 228.6 90.1762 0)
 			(effects
@@
 		(dnp no)
 		(fields_autoplaced yes)
-		(property "Reference" "C1"
+		(property "Reference" "C?"
 			(at 236.22 90.1762 0)
 			(effects
@@
 				)
 			)
+			(project "nzif"
+				(path "/fe42ca2f-2bb8-4d5a-9e84-807788ed632f/d1b276aa-cc76-4829-b01b-98095216e3ce"
+					(reference "C?")
+					(unit 1)
+				)
+			)
 		)
 	)
@@
 		(dnp no)
 		(fields_autoplaced yes)
-		(property "Reference" "#PWR?"
+		(property "Reference" "#PWR0213"
 			(at 105.41 127 0)
 			(effects
@@
 		(dnp no)
 		(fields_autoplaced yes)
-		(property "Reference" "#PWR01"
+		(property "Reference" "#PWR?"
 			(at 208.28 100.33 0)
 			(effects
@@
 				)
 			)
+			(project "nzif"
+				(path "/fe42ca2f-2bb8-4d5a-9e84-807788ed632f/d1b276aa-cc76-4829-b01b-98095216e3ce"
+					(reference "#PWR?")
+					(unit 1)
+				)
+			)
 		)
 	)
@@
 		(on_board yes)
 		(dnp no)
-		(property "Reference" "#PWR?"
+		(property "Reference" "#PWR0210"
 			(at 184.15 160.02 0)
 			(effects
@@
 		(dnp no)
 		(fields_autoplaced yes)
-		(property "Reference" "#PWR?"
+		(property "Reference" "#PWR0206"
 			(at 252.73 154.94 0)
 			(effects
@@
 		(dnp no)
 		(fields_autoplaced yes)
-		(property "Reference" "#PWR?"
+		(property "Reference" "#PWR0215"
 			(at 127 135.89 0)
 			(effects
@@
 		(on_board yes)
 		(dnp no)
-		(property "Reference" "U?"
+		(property "Reference" "U202"
 			(at 215.138 127 0)
 			(effects
@@
 		(dnp no)
 		(fields_autoplaced yes)
-		(property "Reference" "C?"
+		(property "Reference" "C202"
 			(at 186.69 149.8662 0)
 			(effects
@@
 		(dnp no)
 		(fields_autoplaced yes)
-		(property "Reference" "#PWR?"
+		(property "Reference" "#PWR0260"
 			(at 233.68 100.33 0)
 			(effects
@@
 		(dnp no)
 		(fields_autoplaced yes)
-		(property "Reference" "#PWR?"
+		(property "Reference" "#PWR0201"
 			(at 173.99 160.02 0)
 			(effects

Commit message: added small resistor values to ADC inputs
Parts:
- added R1, R2, R3, R4, R5, R6, R7, R8: 10, Resistor_SMD:R_0603_1608Metric_Pad0.98x0.95mm_HandSolder, symbol Device:R_Small_US
- renumbered C209 to C?, C204 to C?, C207 to C?, C201 to C?, C203 to C?, C210 to C?, C208 to C?, C205 to C?, C202 to C?, R201 to R?, R208 to R?, R202 to R?, U201 to U?, U202 to U?
Connections:
- net AIN1N: now also R2.1; no longer U?.32 (AIN1N)
- net AIN1P: now also R1.1; no longer U?.33 (AIN1P)
- net AIN2N: now also R3.1; no longer U?.34 (AIN2N)
- net AIN2P: now also R4.1; no longer U?.35 (AIN2P)
- net AIN3N: now also R5.1; no longer U?.36 (AIN3N)
- net AIN3P: now also R6.1; no longer U?.37 (AIN3P)
- net AIN4N: now also R7.1; no longer U?.38 (AIN4N)
- net AIN4P: now also R8.1; no longer U?.39 (AIN4P)
- new net: R7.2, U?.38 (AIN4N)
- new net: R5.2, U?.36 (AIN3N)
- new net: R4.2, U?.35 (AIN2P)
- new net: R2.2, U?.32 (AIN1N)
- new net: R3.2, U?.34 (AIN2N)
- new net: R8.2, U?.39 (AIN4P)
- new net: R1.2, U?.33 (AIN1P)
- new net: R6.2, U?.37 (AIN3P)

Commit message: added transformer for low band tx
Parts:
- gave numbers to parts that had none: 14
Changed lines of the file:
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@@
 		(dnp no)
 		(fields_autoplaced yes)
-		(property "Reference" "C?"
+		(property "Reference" "C209"
 			(at 107.95 116.8462 0)
 			(effects
@@
 		(dnp no)
 		(fields_autoplaced yes)
-		(property "Reference" "#PWR?"
+		(property "Reference" "#PWR0209"
 			(at 246.38 135.89 0)
 			(effects
@@
 		(dnp no)
 		(fields_autoplaced yes)
-		(property "Reference" "C2"
+		(property "Reference" "C?"
 			(at 243.84 90.1762 0)
 			(effects
@@
 		(dnp no)
 		(fields_autoplaced yes)
-		(property "Reference" "#PWR?"
+		(property "Reference" "#PWR0207"
 			(at 246.38 138.43 0)
 			(effects
@@
 		(dnp no)
 		(fields_autoplaced yes)
-		(property "Reference" "#PWR?"
+		(property "Reference" "#PWR0203"
 			(at 218.44 165.1 0)
 			(effects
@@
 		(dnp yes)
 		(fields_autoplaced yes)
-		(property "Reference" "C?"
+		(property "Reference" "C204"
 			(at 195.58 160.0135 0)
 			(effects
@@
 		(dnp no)
 		(fields_autoplaced yes)
-		(property "Reference" "#PWR?"
+		(property "Reference" "#PWR0205"
 			(at 240.03 173.99 0)
 			(effects
@@
 		(on_board yes)
 		(dnp no)
-		(property "Reference" "U?"
+		(property "Reference" "U201"
 			(at 133.604 113.792 0)
 			(effects
@@
 		(dnp no)
 		(fields_autoplaced yes)
-		(property "Reference" "R7"
+		(property "Reference" "R?"
 			(at 184.15 134.62 90)
 			(effects
@@
 				)
 			)
+			(project "nzif"
+				(path "/fe42ca2f-2bb8-4d5a-9e84-807788ed632f/d1b276aa-cc76-4829-b01b-98095216e3ce"
+					(reference "R?")
+					(unit 1)
+				)
+			)
 		)
 	)
@@
 		(dnp no)
 		(fields_autoplaced yes)
-		(property "Reference" "#PWR?"
+		(property "Reference" "#PWR0204"
 			(at 226.06 100.33 0)
 			(effects
@@
 		(dnp no)
 		(fields_autoplaced yes)
-		(property "Reference" "C?"
+		(property "Reference" "C207"
 			(at 233.68 165.0937 90)
 			(effects
@@
 		(dnp no)
 		(fields_autoplaced yes)
-		(property "Reference" "R5"
+		(property "Reference" "R?"
 			(at 184.15 127 90)
 			(effects
@@
 				)
 			)
+			(project "nzif"
+				(path "/fe42ca2f-2bb8-4d5a-9e84-807788ed632f/d1b276aa-cc76-4829-b01b-98095216e3ce"
+					(reference "R?")
+					(unit 1)
+				)
+			)
 		)
 	)
@@
 		(dnp no)
 		(fields_autoplaced yes)
-		(property "Reference" "#PWR?"
+		(property "Reference" "#PWR0202"
 			(at 248.92 100.33 0)
 			(effects
@@
 		(dnp yes)
 		(fields_autoplaced yes)
-		(property "Reference" "R?"
+		(property "Reference" "R201"
 			(at 195.58 170.1799 0)
 			(effects
@@
 		(dnp no)
 		(fields_autoplaced yes)
-		(property "Reference" "#PWR?"
+		(property "Reference" "#PWR0259"
 			(at 241.3 100.33 0)
 			(effects
@@
 		(dnp no)
 		(fields_autoplaced yes)
-		(property "Reference" "C?"
+		(property "Reference" "C201"
 			(at 176.53 149.8662 0)
 			(effects
@@
 		(on_board yes)
 		(dnp yes)
-		(property "Reference" "C?"
+		(property "Reference" "C203"
 			(at 185.42 165.0935 0)
 			(effects
@@
 		(dnp no)
 		(fields_autoplaced yes)
-		(property "Reference" "R4"
+		(property "Reference" "R?"
 			(at 189.23 116.84 90)
 			(effects
@@
 				)
 			)
+			(project "nzif"
+				(path "/fe42ca2f-2bb8-4d5a-9e84-807788ed632f/d1b276aa-cc76-4829-b01b-98095216e3ce"
+					(reference "R?")
+					(unit 1)
+				)
+			)
 		)
 	)
@@
 		(dnp no)
 		(fields_autoplaced yes)
-		(property "Reference" "C?"
+		(property "Reference" "C210"
 			(at 97.79 116.8462 0)
 			(effects
@@
 		(dnp no)
 		(fields_autoplaced yes)
-		(property "Reference" "C3"
+		(property "Reference" "C?"
 			(at 251.46 90.1762 0)
 			(effects
@@
 		(dnp no)
 		(fields_autoplaced yes)
-		(property "Reference" "R2"
+		(property "Reference" "R?"
 			(at 184.15 111.76 90)
 			(effects
@@
 				)
 			)
+			(project "nzif"
+				(path "/fe42ca2f-2bb8-4d5a-9e84-807788ed632f/d1b276aa-cc76-4829-b01b-98095216e3ce"
+					(reference "R?")
+					(unit 1)
+				)
+			)
 		)
 	)
@@
 		(dnp no)
 		(fields_autoplaced yes)
-		(property "Reference" "R3"
+		(property "Reference" "R?"
 			(at 184.15 119.38 90)
 			(effects
@@
 				)
 			)
+			(project "nzif"
+				(path "/fe42ca2f-2bb8-4d5a-9e84-807788ed632f/d1b276aa-cc76-4829-b01b-98095216e3ce"
+					(reference "R?")
+					(unit 1)
+				)
+			)
 		)
 	)
@@
 		(dnp no)
 		(fields_autoplaced yes)
-		(property "Reference" "R?"
+		(property "Reference" "R208"
 			(at 266.7 139.7 90)
 			(effects
@@
 		(dnp no)
 		(fields_autoplaced yes)
-		(property "Reference" "R8"
+		(property "Reference" "R?"
 			(at 189.23 132.08 90)
 			(effects
@@
 				)
 			)
+			(project "nzif"
+				(path "/fe42ca2f-2bb8-4d5a-9e84-807788ed632f/d1b276aa-cc76-4829-b01b-98095216e3ce"
+					(reference "R?")
+					(unit 1)
+				)
+			)
 		)
 	)
@@
 		(dnp no)
 		(fields_autoplaced yes)
-		(property "Reference" "R?"
+		(property "Reference" "R202"
 			(at 259.08 163.8299 0)
 			(effects
@@
 		(dnp no)
 		(fields_autoplaced yes)
-		(property "Reference" "C4"
+		(property "Reference" "C?"
 			(at 210.82 90.1762 0)
 			(effects
@@
 		(dnp no)
 		(fields_autoplaced yes)
-		(property "Reference" "C?"
+		(property "Reference" "C208"
 			(at 248.92 165.0937 90)
 			(effects
@@
 		(dnp no)
 		(fields_autoplaced yes)
-		(property "Reference" "R1"
+		(property "Reference" "R?"
 			(at 189.23 109.22 90)
 			(effects
@@
 				)
 			)
+			(project "nzif"
+				(path "/fe42ca2f-2bb8-4d5a-9e84-807788ed632f/d1b276aa-cc76-4829-b01b-98095216e3ce"
+					(reference "R?")
+					(unit 1)
+				)
+			)
 		)
 	)
@@
 		(dnp no)
 		(fields_autoplaced yes)
-		(property "Reference" "#PWR?"
+		(property "Reference" "#PWR0208"
 			(at 245.11 173.99 0)
 			(effects
@@
 		(dnp no)
 		(fields_autoplaced yes)
-		(property "Reference" "#PWR?"
+		(property "Reference" "#PWR0258"
 			(at 256.54 173.99 0)
 			(effects
@@
 		(dnp no)
 		(fields_autoplaced yes)
-		(property "Reference" "#PWR?"
+		(property "Reference" "#PWR0214"
 			(at 95.25 127 0)
 			(effects
@@
 		(dnp no)
 		(fields_autoplaced yes)
-		(property "Reference" "C?"
+		(property "Reference" "C205"
 			(at 228.6 90.1762 0)
 			(effects
@@
 		(dnp no)
 		(fields_autoplaced yes)
-		(property "Reference" "C1"
+		(property "Reference" "C?"
 			(at 236.22 90.1762 0)
 			(effects
@@
 		(dnp no)
 		(fields_autoplaced yes)
-		(property "Reference" "R6"
+		(property "Reference" "R?"
 			(at 189.23 124.46 90)
 			(effects
@@
 				)
 			)
+			(project "nzif"
+				(path "/fe42ca2f-2bb8-4d5a-9e84-807788ed632f/d1b276aa-cc76-4829-b01b-98095216e3ce"
+					(reference "R?")
+					(unit 1)
+				)
+			)
 		)
 	)
@@
 		(dnp no)
 		(fields_autoplaced yes)
-		(property "Reference" "#PWR?"
+		(property "Reference" "#PWR0213"
 			(at 105.41 127 0)
 			(effects
@@
 		(dnp no)
 		(fields_autoplaced yes)
-		(property "Reference" "#PWR01"
+		(property "Reference" "#PWR?"
 			(at 208.28 100.33 0)
 			(effects
@@
 		(on_board yes)
 		(dnp no)
-		(property "Reference" "#PWR?"
+		(property "Reference" "#PWR0210"
 			(at 184.15 160.02 0)
 			(effects
@@
 		(dnp no)
 		(fields_autoplaced yes)
-		(property "Reference" "#PWR?"
+		(property "Reference" "#PWR0206"
 			(at 252.73 154.94 0)
 			(effects
@@
 		(dnp no)
 		(fields_autoplaced yes)
-		(property "Reference" "#PWR?"
+		(property "Reference" "#PWR0215"
 			(at 127 135.89 0)
 			(effects
@@
 		(on_board yes)
 		(dnp no)
-		(property "Reference" "U?"
+		(property "Reference" "U202"
 			(at 215.138 127 0)
 			(effects
@@
 		(dnp no)
 		(fields_autoplaced yes)
-		(property "Reference" "C?"
+		(property "Reference" "C202"
 			(at 186.69 149.8662 0)
 			(effects
@@
 		(dnp no)
 		(fields_autoplaced yes)
-		(property "Reference" "#PWR?"
+		(property "Reference" "#PWR0260"
 			(at 233.68 100.33 0)
 			(effects
@@
 		(dnp no)
 		(fields_autoplaced yes)
-		(property "Reference" "#PWR?"
+		(property "Reference" "#PWR0201"
 			(at 173.99 160.02 0)
 			(effects
