File: nzif/dacs.kicad_sch (KiCad schematic)
At the start: 122 parts, among them Q102 FZT951TA, U134 ADAU1962AWBSTZ-RL

Commit message: updated DAC
Parts:
- removed C189, C191, C194, C199, C205, C207, C209, C211, C213, C215: 10n, symbol Device:C_Small_US
- removed C190, C192, C195, C200, C206, C208, C210, C212, C214, C216: .1u, symbol Device:C_Small_US
- removed C221, C222, C223, C224, C235, C236, C237, C238, C247, C248, C249, C250: 2.7n, symbol Device:C_Small_US
- removed C225, C226, C227, C228, C229, C230, C231, C232, C239, C240, C241, C242, C243, C244, C245, C246, C251, C252, C253, C254, C255, C256, C257, C258: 10u, symbol Device:C_Small_US
- removed R167, R168, R169, R170, R171, R172, R173, R174, R184, R185, R186, R187, R188, R189, R190, R191, R200, R201, R202, R203, R204, R205, R206, R207: 237, symbol Device:R_Small_US
- removed R175, R176, R177, R178, R179, R180, R181, R182, R192, R193, R194, R195, R196, R197, R198, R199, R208, R209, R210, R211, R212, R213, R214, R215: 49.9k, symbol Device:R_Small_US
- added C1, C10, C11, C14, C15, C16, C2, C3, C4, C5: 10u, symbol Device:C_Small_US
- added C12, C19, C8: 0.iu, symbol Device:C_Small_US
- added C13, C17, C18, C20, C6, C7, C9: 0.1u, symbol Device:C_Small_US
- added C21: 10n, symbol Device:C_Small_US
- added C22: .1u, symbol Device:C_Small_US
- added R1: 49.9, symbol Device:R_Small_US
- added R10, R11, R12, R13, R2, R3, R4, R5, R6, R7, R8, R9: 100, symbol Device:R_Small_US
- added U2: ADA4807-1, symbol Amplifier_Operational:ADA4807-1
- C?: renamed from C233; value 150p -> 39n
- C?: renamed from C234; value 2.2n -> 2.2n NPO
- renumbered C203 to C?, C220 to C?, C202 to C?, C201 to C?, C196 to C?, C218 to C?, C197 to C?, C193 to C?, C219 to C?, C204 to C?, C217 to C?, C198 to C?, Q102 to Q?, R166 to R?, R183 to R?, U134 to U1
Connections:
- net 2.5: no longer U1.16 (PLLVDD)
- net 2.5V: now also U1.16 (PLLVDD), U1.20 (DVDD), U1.25 (VSUPPLY), U1.29 (DVDD), U1.41 (DVDD), C1.1, C14.1, C15.1, C16.1, C17.1, C18.1, C19.1, C20.1; no longer U1.23 (VSENSE)
- net 3.3V: now also U1.12 (AVDD4), U1.22 (IOVDD), U1.23 (VSENSE), U1.3 (AVDD3), U1.39 (IOVDD), U1.49 (AVDD1), U1.58 (AVDD2), C10.1, C11.1, C12.1, C13.1, C2.1, C3.1, C4.1, C5.1, C6.1, C7.1, C8.1, C9.1; no longer U1.25 (VSUPPLY)
- net AVDD2: no longer U1.58 (AVDD2)
- net AVDD3: no longer U1.12 (AVDD4), U1.3 (AVDD3)
- net GND: now also U1.13 (AGND4), U1.14 (PLLGND), U1.21 (DGND), U1.26 (DGND), U1.30 (DGND), U1.31 (SA1), U1.32 (SA2), U1.40 (DGND), U1.42 (MOSI/ADDR1/SA), U1.45 (SS*/ADDR0/SA), U1.46 (SA_MODE), U1.48 (AGND1), U1.61 (AGND2), U1.80 (AGND3), C1.2, C10.2, C11.2, C12.2, C13.2, C14.2, C15.2, C16.2, C17.2, C18.2, C19.2, C2.2, C20.2, C21.2, C22.2, C3.2, C4.2, C5.2, C6.2, C7.2, C8.2, C9.2, U2.2 (V-); no longer U1.13 (AGND4), U1.14 (PLLGND), U1.21 (DGND), U1.26 (DGND), U1.30 (DGND), U1.31 (SA1), U1.32 (SA2), U1.40 (DGND), U1.42 (MOSI/ADDR1/SA), U1.46 (SA_MODE), U1.48 (AGND1), U1.61 (AGND2), U1.80 (AGND3)
- net MCLK: now also R1.1; no longer U1.17 (MCLKI/XTALI)
- net MISO_SDA: now also U1.43 (MISO/SDA/SA); no longer U1.43 (MISO/SDA/SA)
- net SCLK/SCL: now also U1.44 (SCLK/SCL); no longer U1.44 (SCLK/SCL)
- net TDM1_SDIN_DAC: now also U1.37 (DSDATA2); no longer U1.38 (DSDATA1)
- net VDRIVE: now also U1.24 (VDRIVE); no longer U1.24 (VDRIVE), U1.45 (SS*/ADDR0/SA)
- net at C?.1, C?.1: now also U1.62 (CM), U2.3 (+); no longer U1.62 (CM)
- net at C?.1, C?.1: now also U1.15 (LF); no longer U1.15 (LF)
- net at C?.1: now also U1.1 (DAC_BIAS3); no longer U1.1 (DAC_BIAS3)
- net at C?.1: now also U1.59 (DAC_BIAS1); no longer U1.59 (DAC_BIAS1)
- net at C?.1, C?.1: now also U1.63 (TS_REF); no longer U1.63 (TS_REF)
- net at C?.1: now also U1.2 (DAC_BIAS4); no longer U1.2 (DAC_BIAS4)
- net at C?.1: now also U1.60 (DAC_BIAS2); no longer U1.60 (DAC_BIAS2)
- removed net AVDD1: U1.49 (AVDD1)
- removed net BCLK_OUT1: U1.27 (DBCLK)
- removed net DAC10N: U1.74 (DAC10P)
- removed net DAC10P: U1.75 (DAC10N)
- removed net DAC11N: U1.76 (DAC11P)
- removed net DAC11P: U1.77 (DAC11N)
- removed net DAC12N: U1.78 (DAC12P)
- removed net DAC12P: U1.79 (DAC12N)
- removed net DAC1N: U1.51 (DAC1N)
- removed net DAC1P: U1.50 (DAC1P)
- removed net DAC2N: U1.52 (DAC2P)
- removed net DAC2P: U1.53 (DAC2N)
- removed net DAC3N: U1.55 (DAC3N)
- removed net DAC3P: U1.54 (DAC3P)
- removed net DAC4N: U1.56 (DAC4P)
- removed net DAC4P: U1.57 (DAC4N)
- removed net DAC5N: U1.65 (DAC5N)
- removed net DAC5P: U1.64 (DAC5P)
- removed net DAC6N: U1.66 (DAC6P)
- removed net DAC6P: U1.67 (DAC6N)
- removed net DAC7N: U1.69 (DAC7N)
- removed net DAC7P: U1.68 (DAC7P)
- removed net DAC8N: U1.70 (DAC8P)
- removed net DAC8P: U1.71 (DAC8N)
- removed net DAC9N: U1.73 (DAC9N)
- removed net DAC9P: U1.72 (DAC9P)
- removed net DVDD: U1.20 (DVDD), U1.29 (DVDD), U1.41 (DVDD)
- removed net IOVDD: U1.22 (IOVDD), U1.39 (IOVDD)
- removed net LRCLK_OUT1: U1.28 (DLRCLK)
- new net: R3.1, U1.52 (DAC2P)
- new net: R11.1, U1.74 (DAC10P)
- new net: C21.1, C22.1, U2.6 (V+)
- new net: R1.2, U1.17 (MCLKI/XTALI)
- new net: R2.1, U1.50 (DAC1P)
- new net: R4.1, U1.54 (DAC3P)
- new net: R5.1, U1.56 (DAC4P)
- new net: R6.1, U1.64 (DAC5P)
- new net: R7.1, U1.66 (DAC6P)
- new net: R8.1, U1.68 (DAC7P)
- new net: R9.1, U1.70 (DAC8P)
- new net: R10.1, U1.72 (DAC9P)
- new net: R12.1, U1.76 (DAC11P)
- new net: R13.1, U1.78 (DAC12P)
- new net: U1.10 (NC), U1.11 (NC), U1.4 (NC), U1.5 (NC), U1.6 (NC), U1.7 (NC), U1.8 (NC), U1.9 (NC)
- new net DAC_CM_1.5V: U2.1, U2.4 (-)
- new net DAC_MONITOR0: R10.2
- new net DAC_MONITOR1: R11.2
- new net DAC_MONITOR2: R12.2
- new net DAC_MONITOR3: R13.2
- new net DAC_P0: R2.2
- new net DAC_P135: R5.2
- new net DAC_P180: R6.2
- new net DAC_P225: R7.2
- new net DAC_P270: R8.2
- new net DAC_P315: R9.2
- new net DAC_P45: R3.2
- new net DAC_P90: R4.2
- new net DBCLK: U1.27 (DBCLK)
- new net DLRCLK: U1.28 (DLRCLK)
- no-connect marks 7 -> 20
Other:
- moved on the sheet: C?, Q?, R?
