File: nzif/dacs.kicad_sch (KiCad schematic)
At the start: 63 parts, among them Q601 FZT951TA, U601 ADAU1962AWBSTZ-RL, U602 ADA4807-1

Commit message: erc updates
Parts:
- R601: value 1k -> 1.5k
Other:
- note added: "check jumpers"
Changed lines of the file:
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@@
 		(company "Andy McCann KA3KAF and Doug McCann KA3KAG")
 	)
+	(text "check jumpers"
+		(exclude_from_sim no)
+		(at 78.74 131.318 0)
+		(effects
+			(font
+				(size 1.27 1.27)
+			)
+		)
+	)
 	(text "DAC_Out_9x to 12x go to a header on the top sheet"
 		(exclude_from_sim no)
@@
 	)
 	(junction
-		(at 72.39 147.32)
-		(diameter 0)
-		(color 0 0 0 0)
-	)
-	(junction
 		(at 198.12 247.65)
 		(diameter 0)
@@
 	)
 	(junction
+		(at 72.39 147.32)
+		(diameter 0)
+		(color 0 0 0 0)
+	)
+	(junction
 		(at 123.19 152.4)
 		(diameter 0)
@@
 	(wire
 		(pts
-			(xy 72.39 147.32) (xy 92.71 147.32)
+			(xy 67.31 147.32) (xy 72.39 147.32)
 		)
 		(stroke
@@
 	(wire
 		(pts
+			(xy 72.39 147.32) (xy 92.71 147.32)
+		)
+		(stroke
+			(width 0)
+			(type default)
+		)
+	)
+	(wire
+		(pts
 			(xy 81.28 157.48) (xy 92.71 157.48)
 		)
@@
 	(wire
 		(pts
-			(xy 67.31 147.32) (xy 72.39 147.32)
-		)
-		(stroke
-			(width 0)
-			(type default)
-		)
-	)
-	(wire
-		(pts
 			(xy 243.84 48.26) (xy 306.07 48.26)
 		)
@@
 		(fields_autoplaced yes)
 		(property "Reference" "R601"
-			(at 111.76 148.5899 0)
+			(at 116.84 148.5899 0)
 			(show_name no)
 			(do_not_autoplace no)
@@
 					(size 1.27 1.27)
 				)
-				(justify right)
+				(justify left)
 			)
 		)
-		(property "Value" "1k"
-			(at 111.76 151.1299 0)
+		(property "Value" "1.5k"
+			(at 116.84 151.1299 0)
 			(show_name no)
 			(do_not_autoplace no)
@@
 					(size 1.27 1.27)
 				)
-				(justify right)
+				(justify left)
 			)
 		)
@@
 	)
 	(symbol
-		(lib_id "power:PWR_FLAG")
-		(at 72.39 147.32 0)
+		(lib_id "Device:C_Small_US")
+		(at 224.79 242.57 0)
+		(mirror y)
 		(unit 1)
 		(body_style 1)
@@
 		(dnp no)
 		(fields_autoplaced yes)
-		(property "Reference" "#FLG01212"
-			(at 72.39 145.415 0)
-			(hide yes)
+		(property "Reference" "C626"
+			(at 227.33 241.4269 0)
 			(show_name no)
 			(do_not_autoplace no)
@@
 					(size 1.27 1.27)
 				)
+				(justify right)
 			)
 		)
-		(property "Value" "PWR_FLAG"
-			(at 72.39 142.24 0)
+		(property "Value" "0.1u"
+			(at 227.33 243.9669 0)
 			(show_name no)
 			(do_not_autoplace no)
@@
 					(size 1.27 1.27)
 				)
+				(justify right)
 			)
 		)
 		(property "Footprint" ""
-			(at 72.39 147.32 0)
+			(at 224.79 242.57 0)
 			(hide yes)
 			(show_name no)
@@
 		)
 		(property "Datasheet" ""
-			(at 72.39 147.32 0)
+			(at 224.79 242.57 0)
 			(hide yes)
 			(show_name no)
@@
 			)
 		)
-		(property "Description" "Special symbol for telling ERC where power comes from"
-			(at 72.39 147.32 0)
+		(property "Description" "capacitor, small US symbol"
+			(at 224.79 242.57 0)
+			(hide yes)
+			(show_name no)
+			(do_not_autoplace no)
+			(effects
+				(font
+					(size 1.27 1.27)
+				)
+			)
+		)
+		(property "Digikey Part #" ""
+			(at 224.79 242.57 0)
 			(hide yes)
 			(show_name no)
@@
 		(pin "1"
 		)
+		(pin "2"
+		)
 		(instances
+			(project "dacs"
+				(path "/2de56439-3342-4514-bfd7-22b434f17500"
+					(reference "C20")
+					(unit 1)
+				)
+			)
 			(project "nzif"
 				(path "/fe42ca2f-2bb8-4d5a-9e84-807788ed632f/1097e363-2947-4914-97f0-a09e0bb38c3a"
-					(reference "#FLG01212")
+					(reference "C626")
 					(unit 1)
 				)
@@
 	)
 	(symbol
-		(lib_id "Device:C_Small_US")
-		(at 224.79 242.57 0)
-		(mirror y)
+		(lib_id "power:PWR_FLAG")
+		(at 72.39 147.32 180)
 		(unit 1)
 		(body_style 1)
@@
 		(dnp no)
 		(fields_autoplaced yes)
-		(property "Reference" "C626"
-			(at 227.33 241.4269 0)
+		(property "Reference" "#FLG01212"
+			(at 72.39 149.225 0)
+			(hide yes)
 			(show_name no)
 			(do_not_autoplace no)
@@
 					(size 1.27 1.27)
 				)
-				(justify right)
 			)
 		)
-		(property "Value" "0.1u"
-			(at 227.33 243.9669 0)
+		(property "Value" "PWR_FLAG"
+			(at 72.39 152.4 0)
 			(show_name no)
 			(do_not_autoplace no)
@@
 					(size 1.27 1.27)
 				)
-				(justify right)
 			)
 		)
 		(property "Footprint" ""
-			(at 224.79 242.57 0)
+			(at 72.39 147.32 0)
 			(hide yes)
 			(show_name no)
@@
 		)
 		(property "Datasheet" ""
-			(at 224.79 242.57 0)
-			(hide yes)
-			(show_name no)
-			(do_not_autoplace no)
-			(effects
-				(font
-					(size 1.27 1.27)
-				)
-			)
-		)
-		(property "Description" "capacitor, small US symbol"
-			(at 224.79 242.57 0)
+			(at 72.39 147.32 0)
 			(hide yes)
 			(show_name no)
@@
 			)
 		)
-		(property "Digikey Part #" ""
-			(at 224.79 242.57 0)
+		(property "Description" "Special symbol for telling ERC where power comes from"
+			(at 72.39 147.32 0)
 			(hide yes)
 			(show_name no)
@@
 		(pin "1"
 		)
-		(pin "2"
-		)
 		(instances
-			(project "dacs"
-				(path "/2de56439-3342-4514-bfd7-22b434f17500"
-					(reference "C20")
-					(unit 1)
-				)
-			)
 			(project "nzif"
 				(path "/fe42ca2f-2bb8-4d5a-9e84-807788ed632f/1097e363-2947-4914-97f0-a09e0bb38c3a"
-					(reference "C626")
+					(reference "#FLG01212")
 					(unit 1)
 				)
