File: nzif/rx_driver_amps.kicad_sch (KiCad schematic)
At the start: 32 parts, among them U2 ADA4945-1, U201 ADA4945-1, U7 LT5400BCMS8E-8-TRPBF, U8 LT5400BCMS8E-8-TRPBF

Commit message: Update Rx driver amps schematic
Parts:
- removed C10, C11: 180p, symbol Device:C_Small
- removed C3, C6: 10u, Capacitor_SMD:C_0603_1608Metric_Pad1.08x0.95mm_HandSolder, symbol Device:C_Small
- removed C4, C5, C7, C8, C9: 0.1u, Capacitor_SMD:C_0603_1608Metric_Pad1.08x0.95mm_HandSolder, symbol Device:C_Small
- removed R2: 3.4k, Resistor_SMD:R_0603_1608Metric_Pad0.98x0.95mm_HandSolder, symbol Device:R_Small_US
- removed R3, R6: 9.53k, Resistor_SMD:R_0603_1608Metric_Pad0.98x0.95mm_HandSolder, symbol Device:R_Small_US
- removed R4, R5: 10k, Resistor_SMD:R_0603_1608Metric_Pad0.98x0.95mm_HandSolder, symbol Device:R_Small_US
- removed U2: ADA4945-1, nzif_footprints:LFCSP16_ADA4945-1ACPZ-R2_ADI, symbol nzif_radio_symbol_library:ADA4945-1
- removed U8: LT5400BCMS8E-8-TRPBF, nzif_footprints:MSOP-8_MS_LIT, symbol nzif_radio_symbol_library:LT5400BCMS8E-8-TRPBF
- renumbered C210 to C?, C215 to C?, C211 to C?, C214 to C?, C209 to C?, C213 to C?, C212 to C?, R210 to R?, R209 to R?, R211 to R?, R212 to R?, U201 to U?
Other:
- moved on the sheet: C1, C2, C?, R1, R?, U7, U?

Commit message: updated FDAs
Parts:
- added C10, C11, C19, C20, C28, C29: 180p, symbol Device:C_Small
- added C12, C15, C21, C24, C3, C6: 10u, Capacitor_SMD:C_0603_1608Metric_Pad1.08x0.95mm_HandSolder, symbol Device:C_Small
- added C13, C14, C16, C17, C18, C22, C23, C25, C26, C27, C4, C5, C7, C8, C9: 0.1u, Capacitor_SMD:C_0603_1608Metric_Pad1.08x0.95mm_HandSolder, symbol Device:C_Small
- added R10, R12, R17, R19, R24, R5: 9.53k, Resistor_SMD:R_0603_1608Metric_Pad0.98x0.95mm_HandSolder, symbol Device:R_Small_US
- added R11, R18, R4: 3.4k, Resistor_SMD:R_0603_1608Metric_Pad0.98x0.95mm_HandSolder, symbol Device:R_Small_US
- added R13, R14, R2, R20, R21, R3, R6, R7: 1k, symbol Device:R_Small_US
- added R15, R16, R22, R23, R8, R9: 10k, Resistor_SMD:R_0603_1608Metric_Pad0.98x0.95mm_HandSolder, symbol Device:R_Small_US
- added U1, U10, U3, U6: ADG884xCP, Package_CSP:LFCSP-WD-10-1EP_3x3mm_P0.5mm_EP1.64x2.38mm, symbol Analog_Switch:ADG884xCP
- added U11, U4, U8: ADA4945-1, nzif_footprints:LFCSP16_ADA4945-1ACPZ-R2_ADI, symbol nzif_radio_symbol_library:ADA4945-1
- added U2, U5, U9: LT5400BCMS8E-8-TRPBF, nzif_footprints:MSOP-8_MS_LIT, symbol nzif_radio_symbol_library:LT5400BCMS8E-8-TRPBF
- C1, C2: now not fitted
Connections:
- net P0_SW+ is gone; now on net P0_IN+: U7.3 (R3)
- net P0_SW- is gone; now on net P0_IN-: U7.2 (R2)
- net +6.5V: now also C12.1, C13.1, C14.1, C21.1, C22.1, C23.1, C3.1, C4.1, C5.1, R11.1, R15.2, R18.1, R22.2, R4.1, R8.2, U11.5 (MODE), U11.6 (+VS), U11.7 (+VS), U4.5 (MODE), U4.6 (+VS), U4.7 (+VS), U8.5 (MODE), U8.6 (+VS), U8.7 (+VS)
- net +VCLAMP: now also R11.2, R12.1, R18.2, R19.1, R4.2, R5.1, U11.8 (+VCLAMP), U4.8 (+VCLAMP), U8.8 (+VCLAMP)
- net -3.5V: now also C15.1, C17.1, C18.1, C24.1, C26.1, C27.1, C6.1, C8.1, C9.1, R16.1, R23.1, R9.1, U11.14 (-VS), U11.15 (-VS), U11.17 (-VS), U4.14 (-VS), U4.15 (-VS), U4.17 (-VS), U8.14 (-VS), U8.15 (-VS), U8.17 (-VS)
- net -VCLAMP: now also R10.1, R16.2, R17.1, R23.2, R24.1, R9.2, U11.13 (-VCLAMP), U4.13 (-VCLAMP), U8.13 (-VCLAMP)
- net GND: now also C12.2, C13.2, C14.2, C15.2, C16.2, C17.2, C18.2, C21.2, C22.2, C23.2, C24.2, C25.2, C26.2, C27.2, C3.2, C4.2, C5.2, C6.2, C7.2, C8.2, C9.2, R10.2, R12.2, R17.2, R19.2, R24.2, R5.2, U11.16 (DGND), U4.16 (DGND), U8.16 (DGND)
- net P0_FB+: now also U1.9 (D2); no longer U7.1 (R1)
- net P0_FB-: now also U1.3 (D1); no longer U7.4 (R4)
- net P0_IN+: now also R2.1
- net P0_IN-: now also R21.1, R3.1
- net VREF_BUF: now also C16.1, C25.1, C7.1, U11.9 (VOCM), U4.9 (VOCM), U8.9 (VOCM)
- new net: R20.2, U10.2 (S1A)
- new net: U10.11 (GND), U10.6 (GND)
- new net: R21.2, U10.7 (S2B)
- new net: R22.1, U11.12 (~{DISABLE})
- new net: R2.2, U1.2 (S1A)
- new net: R15.1, U8.12 (~{DISABLE})
- new net: R6.2, U3.2 (S1A)
- new net: R7.2, U3.7 (S2B)
- new net: U3.11 (GND), U3.6 (GND)
- new net: U6.11 (GND), U6.6 (GND)
- new net: R13.2, U6.2 (S1A)
- new net: R14.2, U6.7 (S2B)
- new net: U1.11 (GND), U1.6 (GND)
- new net: R3.2, U1.7 (S2B)
- new net: R8.1, U4.12 (~{DISABLE})
- new net LT5400_p1: U1.10 (S2A), U10.10 (S2A), U2.1 (R1), U3.10 (S2A), U5.1 (R1), U6.10 (S2A), U7.1 (R1), U9.1 (R1)
- new net LT5400_p4: U1.5 (S1B), U10.5 (S1B), U2.4 (R4), U3.5 (S1B), U5.4 (R4), U6.5 (S1B), U7.4 (R4), U9.4 (R4)
- new net P135_FDA+: U11.10 (+OUT)
- new net P135_FDA-: U11.11 (-OUT)
- new net P135_IN+: U9.3 (R3)
- new net P135_IN-: U9.2 (R2)
- new net P1_FB+: C20.1, U6.9 (D2), U8.4 (+FB)
- new net P1_FB-: C19.1, U6.3 (D1), U8.1 (-FB)
- new net P1_IN+: C19.2, R13.1, U5.5 (R4), U5.6 (R3), U8.2 (+IN)
- new net P1_IN-: C20.2, R14.1, U5.7 (R2), U5.8 (R1), U8.3 (-IN)
- new net P2_FB+: C11.1, U3.9 (D2), U4.4 (+FB)
- new net P2_FB-: C10.1, U3.3 (D1), U4.1 (-FB)
- new net P2_IN+: C10.2, R6.1, U2.5 (R4), U2.6 (R3), U4.2 (+IN)
- new net P2_IN-: C11.2, R7.1, U2.7 (R2), U2.8 (R1), U4.3 (-IN)
- new net P3_FB+: C29.1, U10.9 (D2), U11.4 (+FB)
- new net P3_FB-: C28.1, U10.3 (D1), U11.1 (-FB)
- new net P3_IN+: C28.2, R20.1, U11.2 (+IN), U9.5 (R4), U9.6 (R3)
- new net P3_IN-: C29.2, U11.3 (-IN), U9.7 (R2), U9.8 (R1)
- new net P45_FDA+: U8.10 (+OUT)
- new net P45_FDA-: U8.11 (-OUT)
- new net P45_IN+: U5.3 (R3)
- new net P45_IN-: U5.2 (R2)
- new net P90_FDA+: U4.10 (+OUT)
- new net P90_FDA-: U4.11 (-OUT)
- new net P90_IN+: U2.3 (R3)
- new net P90_IN-: U2.2 (R2)
- new net uc_gain_select_0: U1.4 (IN1), U1.8 (IN2), U10.4 (IN1), U10.8 (IN2), U3.4 (IN1), U3.8 (IN2), U6.4 (IN1), U6.8 (IN2)
Other:
- note added: "-VCLAMP set to -1.7V"
- note removed: "-VCLAMP set to -2.2V"
- note removed: "This should be 9x"
- moved on the sheet: C?, R1, R?, U7, U?

Commit message: reordered sheets - annotate sheets - set all to no sim
Parts:
- gave numbers to parts that had none: 12
- renumbered C12 to C110, C13 to C112, C14 to C114, C15 to C116, C16 to C119, C17 to C120, C18 to C122, C1 to C123, C2 to C124, C19 to C125, C20 to C126, C21 to C127, C22 to C128, C23 to C129, C3 to C130, C4 to C131, C5 to C132, C24 to C133, C25 to C134, C26 to C135, C6 to C136, C27 to C137, C7 to C138, C8 to C139, C28 to C140, C29 to C141, C9 to C142, C10 to C143, C11 to C144, R11 to R106, R12 to R107, R2 to R108, R3 to R109, R13 to R110, R14 to R111, R1 to R112, R15 to R113, R16 to R116, R17 to R117, R18 to R118, R19 to R119, R20 to R120, R21 to R121, R4 to R122, R5 to R123, R22 to R124, R6 to R125, R7 to R126, R8 to R127, R23 to R128, R24 to R129, R9 to R130, R10 to R131, U7 to U117, U5 to U118, U1 to U119, U6 to U120, U8 to U122, U9 to U123, U2 to U124, U10 to U125, U3 to U126, U11 to U127, U4 to U128

Commit message: add supplies for switches on driver amp sheet
Parts:
- added C211, C214, C216, C222: 0.1u, Capacitor_SMD:C_0603_1608Metric_Pad1.08x0.95mm_HandSolder, symbol Device:C_Small
- added C212, C213, C215, C221: 10u, Capacitor_SMD:C_0603_1608Metric_Pad1.08x0.95mm_HandSolder, symbol Device:C_Small
Connections:
- net GND: now also U119.11 (GND), U119.6 (GND), U120.11 (GND), U120.6 (GND), U125.11 (GND), U125.6 (GND), U126.11 (GND), U126.6 (GND), C211.2, C212.2, C213.2, C214.2, C215.2, C216.2, C221.2, C222.2
- net 3.3V: now reaches U125.1 (VDD)
- net 3.3V: now also U119.1 (VDD), U120.1 (VDD), U126.1 (VDD), C211.1, C212.1, C213.1, C214.1, C215.1, C216.1, C221.1, C222.1
Other:
- moved on the sheet: R108, R109, R110, R111, R120, R121, U119, U120, U125

Commit message: added control signals
Parts:
- renumbered C123 to C1, C143 to C10, C144 to C11, C110 to C12, C112 to C13, C114 to C14, C116 to C15, C119 to C16, C120 to C17, C122 to C18, C125 to C19, C124 to C2, C126 to C20, C127 to C21, C128 to C22, C129 to C23, C133 to C24, C134 to C25, C135 to C26, C137 to C27, C140 to C28, C141 to C29, C130 to C3, C131 to C4, C132 to C5, C136 to C6, C138 to C7, C139 to C8, C142 to C9, C109 to C?, C111 to C?, C221 to C?, C115 to C?, C117 to C?, C222 to C?, C215 to C?, C214 to C?, C113 to C?, C213 to C?, C211 to C?, C216 to C?, C121 to C?, C118 to C?, C212 to C?, R112 to R1, R131 to R10, R106 to R11, R107 to R12, R110 to R13, R111 to R14, R113 to R15, R116 to R16, R117 to R17, R118 to R18, R119 to R19, R108 to R2, R120 to R20, R121 to R21, R124 to R22, R128 to R23, R129 to R24, R109 to R3, R122 to R4, R123 to R5, R125 to R6, R126 to R7, R127 to R8, R130 to R9, R105 to R?, R104 to R?, R114 to R?, R115 to R?, U119 to U1, U125 to U10, U127 to U11, U124 to U2, U126 to U3, U128 to U4, U118 to U5, U120 to U6, U117 to U7, U122 to U8, U123 to U9, U121 to U?
Connections:
- net uc_gain_select_0 renamed uC_GAIN_SEL

Commit message: Fix op amps to be correct units
Parts:
- gave numbers to parts that had none: 20
- renumbered C12 to C110, C13 to C112, C14 to C114, C15 to C116, C16 to C119, C17 to C120, C18 to C122, C1 to C123, C2 to C124, C19 to C125, C20 to C126, C21 to C127, C22 to C128, C23 to C129, C3 to C130, C4 to C131, C5 to C132, C24 to C133, C25 to C134, C26 to C135, C6 to C136, C27 to C137, C7 to C138, C8 to C139, C28 to C140, C29 to C141, C9 to C142, C10 to C143, C11 to C144, R11 to R106, R12 to R107, R2 to R108, R3 to R109, R13 to R110, R14 to R111, R1 to R112, R15 to R113, R16 to R116, R17 to R117, R18 to R118, R19 to R119, R20 to R120, R21 to R121, R4 to R122, R5 to R123, R22 to R124, R6 to R125, R7 to R126, R8 to R127, R23 to R128, R24 to R129, R9 to R130, R10 to R131, U7 to U117, U5 to U118, U1 to U119, U6 to U120, U8 to U122, U9 to U123, U2 to U124, U10 to U125, U3 to U126, U11 to U127, U4 to U128
