File: nzif/microcontroller.kicad_sch (KiCad schematic)
At the start: 15 parts, among them U1002 MCP23017_SO, U1203 AD5593R

Commit message: update to clocktree
Connections:
- net SWIO_2 renamed RX_INIT_CLK
- net SWIO_3 renamed TX_INIT_CLK
Changed lines of the file:
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@@
 		)
 	)
-	(hierarchical_label "SWIO_2"
+	(hierarchical_label "RX_INIT_CLK"
 		(shape input)
 		(at 105.41 177.8 0)
@@
 		)
 	)
-	(hierarchical_label "SWIO_3"
+	(hierarchical_label "TX_INIT_CLK"
 		(shape input)
 		(at 105.41 180.34 0)

Commit message: updated clocktree and associated section of README.md
Connections:
- net SWIO_1 renamed PHASE_SEL_8
Changed lines of the file:
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@@
 		)
 	)
-	(hierarchical_label "SWIO_1"
+	(hierarchical_label "PHASE_SEL_8"
 		(shape input)
 		(at 105.41 175.26 0)

Commit message: erc improvements
Changed lines of the file:
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@@
-		)
-	)
-	(label "3.3V"
-		(at 171.45 173.99 0)
-		(effects
-			(font
-				(size 1.27 1.27)
-			)
-			(justify left bottom)
 		)
 	)

Commit message: fixing erc errors
Parts:
- U1002: symbol Interface_Expansion:MCP23017_SO -> nzif_radio_symbol_library:MCP23017_SO
Changed lines of the file:
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@@
 	)
 	(symbol
-		(lib_id "Interface_Expansion:MCP23017_SO")
+		(lib_id "nzif_radio_symbol_library:MCP23017_SO")
 		(at 215.9 217.17 0)
 		(unit 1)

Commit message: added footprints for Rs and Cs
Parts:
- C1004, C1005, C1006, C1007, C1008, C1009, C1010, C1016, C1017: footprint (none) -> Capacitor_SMD:C_0402_1005Metric_Pad0.74x0.62mm_HandSolder
- R1212, R1213, R1219: footprint (none) -> Resistor_SMD:R_0402_1005Metric_Pad0.72x0.64mm_HandSolder
Changed lines of the file:
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@@
 			)
 		)
-		(property "Footprint" ""
+		(property "Footprint" "Resistor_SMD:R_0402_1005Metric_Pad0.72x0.64mm_HandSolder"
 			(at 190.5 138.43 0)
 			(hide yes)
@@
 			)
 		)
-		(property "Footprint" ""
+		(property "Footprint" "Resistor_SMD:R_0402_1005Metric_Pad0.72x0.64mm_HandSolder"
 			(at 130.81 123.19 0)
 			(hide yes)
@@
 			)
 		)
-		(property "Footprint" ""
+		(property "Footprint" "Capacitor_SMD:C_0402_1005Metric_Pad0.74x0.62mm_HandSolder"
 			(at 215.9 52.07 0)
 			(hide yes)
@@
 			)
 		)
-		(property "Footprint" ""
+		(property "Footprint" "Capacitor_SMD:C_0402_1005Metric_Pad0.74x0.62mm_HandSolder"
 			(at 205.74 180.34 0)
 			(hide yes)
@@
 			)
 		)
-		(property "Footprint" ""
+		(property "Footprint" "Capacitor_SMD:C_0402_1005Metric_Pad0.74x0.62mm_HandSolder"
 			(at 251.46 115.57 0)
 			(hide yes)
@@
 			)
 		)
-		(property "Footprint" ""
+		(property "Footprint" "Capacitor_SMD:C_0402_1005Metric_Pad0.74x0.62mm_HandSolder"
 			(at 204.47 52.07 0)
 			(hide yes)
@@
 			)
 		)
-		(property "Footprint" ""
+		(property "Footprint" "Capacitor_SMD:C_0402_1005Metric_Pad0.74x0.62mm_HandSolder"
 			(at 66.04 154.94 0)
 			(hide yes)
@@
 			)
 		)
-		(property "Footprint" ""
+		(property "Footprint" "Capacitor_SMD:C_0402_1005Metric_Pad0.74x0.62mm_HandSolder"
 			(at 48.26 184.15 0)
 			(hide yes)
@@
 			)
 		)
-		(property "Footprint" ""
+		(property "Footprint" "Capacitor_SMD:C_0402_1005Metric_Pad0.74x0.62mm_HandSolder"
 			(at 55.88 154.94 0)
 			(hide yes)
@@
 			)
 		)
-		(property "Footprint" ""
+		(property "Footprint" "Resistor_SMD:R_0402_1005Metric_Pad0.72x0.64mm_HandSolder"
 			(at 146.05 132.08 0)
 			(hide yes)
@@
 			)
 		)
-		(property "Footprint" ""
+		(property "Footprint" "Capacitor_SMD:C_0402_1005Metric_Pad0.74x0.62mm_HandSolder"
 			(at 195.58 180.34 0)
 			(hide yes)
@@
 			)
 		)
-		(property "Footprint" ""
+		(property "Footprint" "Capacitor_SMD:C_0402_1005Metric_Pad0.74x0.62mm_HandSolder"
 			(at 87.63 154.94 0)
 			(hide yes)
@@
 		)
 	)
-	(embedded_fonts no)
 )
