File: nzif/nzif.kicad_pcb (KiCad board)
At the start: 2 copper layers, 619 parts, among them J101 Rx, J102 Tx, J105 Conn_02x05_Odd_Even, J110 6V, J1204 AUX, J1205 AUX, J1206 AUX, J1207 GPIOS, J1208 SKR, J1209 TRRS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

Commit message: added footprints for L that goes with LT8330
Parts:
- added L1201: 8018_74489430027, nzif_footprints:L_Wurth_WE-TDC-8018, F.Cu at (-60.7, 172.1)
- added L1202: 8018_74489430027, nzif_footprints:L_Wurth_WE-TDC-8018, F.Cu at (-50.2, 172.1)
